File: 02_BMS.sch (KiCad schematic (older format))
At the start: 0 parts

Commit message: BMS fertig, Charger fertig, Amplifier fertig. TODO: Charge vs Discharge LiPo wie machen sachen
Parts:
- added C? (x7): 1uF, symbol Device:C_Small
- added C?: 10uF, symbol Device:C_Small
- added C? (x3): 0.1uF, symbol Device:C_Small
- added C?: 4.7uF, symbol Device:C_Small
- added D?: D_Small, symbol Device:D_Small
- added J?: Screw_Terminal_01x07, symbol Connector:Screw_Terminal_01x07
- added Q? (x2): Q_NMOS_DGS, symbol Device:Q_NMOS_DGS
- added Q?: Q_PMOS_DGS, symbol Device:Q_PMOS_DGS
- added R? (x8): 100R, symbol Device:R_Small
- added R?: 0.01R, symbol Device:R_Small
- added R? (x4): 1M, symbol Device:R_Small
- added R?: 10K DNP, symbol Device:R_Small
- added U?: BQ76920, symbol Battery_Management:BQ76920
Connections:
- net labels added: +BATT, ALERT_BQ76920, BOOT_BQ76920, GND, GNDPWR, LDO_BQ76920, R_Therm, SCL, SDA
- wire segments 0 -> 115
Other:
- note added: "10-kΩ NTC 103AT"
- note added: "I2C-Address: 0x08\n"
- note added: "PCH FET"
- note added: "Rsns: 100mV bei 10A = 10mΩ"
