File: AudioProcessor.sch (KiCad schematic (older format))
At the start: 28 parts, among them J601 AudioJack3_Ground, J602 Conn_02x01, U601 XC6216C, U602 TDA7418

Commit message: fast alle footprints herausgesucht. Spulen typen rausgesucht: Bourns spulen
Parts:
- removed J601: AudioJack3_Ground, symbol Connector:AudioJack3_Ground
- removed R610: 47K, symbol Device:R_Small
- added J601: SJ1-3533 CUI Devices, Connector_Audio:Jack_3.5mm_CUI_SJ1-3533NG_Horizontal, symbol Connector:AudioJack2_Ground
- C601, C602, C603, C604, C605, C606, C607, C608, C609, C610, C611, C612: footprint (none) -> Capacitor_SMD:C_0603_1608Metric_Pad1.05x0.95mm_HandSolder
- J602: footprint (none) -> Connector_PinHeader_2.54mm:PinHeader_1x02_P2.54mm_Vertical
- R601, R602, R603, R604, R605, R606, R607, R608, R609, R611, R612: footprint (none) -> Resistor_SMD:R_0603_1608Metric_Pad1.05x0.95mm_HandSolder
- U601: footprint (none) -> Package_TO_SOT_SMD:SOT-23-5_HandSoldering
- U602: footprint (none) -> Package_SO:SOIC-18W_7.5x11.6mm_P1.27mm
Connections:
- net labels removed: AUX_DETECT
- wire segments 69 -> 66
Changed lines of the file:
@@
 F 0 "U602" H 7450 4850 50  0000 C CNN
 F 1 "TDA7418" H 7450 4500 50  0000 C CNN
-F 2 "" H 7250 4700 50  0001 C CNN
+F 2 "Package_SO:SOIC-18W_7.5x11.6mm_P1.27mm" H 7250 4700 50  0001 C CNN
 F 3 "" H 7250 4700 50  0001 C CNN
 	1    7450 4650
@@
 F 0 "C612" H 6850 3600 50  0000 L CNN
 F 1 "100nF" H 6800 3500 50  0000 L CNN
-F 2 "" H 7200 3550 50  0001 C CNN
+F 2 "Capacitor_SMD:C_0603_1608Metric_Pad1.05x0.95mm_HandSolder" H 7200 3550 50  0001 C CNN
 F 3 "~" H 7200 3550 50  0001 C CNN
 	1    7200 3550
@@
 F 0 "C603" V 4700 4250 50  0000 L CNN
 F 1 "1uF" V 4800 4250 50  0000 L CNN
-F 2 "" H 4950 4300 50  0001 C CNN
+F 2 "Capacitor_SMD:C_0603_1608Metric_Pad1.05x0.95mm_HandSolder" H 4950 4300 50  0001 C CNN
 F 3 "~" H 4950 4300 50  0001 C CNN
 	1    4950 4300
@@
 F 0 "C605" V 4950 4300 50  0000 L CNN
 F 1 "1uF" V 5050 4300 50  0000 L CNN
-F 2 "" H 5150 4450 50  0001 C CNN
+F 2 "Capacitor_SMD:C_0603_1608Metric_Pad1.05x0.95mm_HandSolder" H 5150 4450 50  0001 C CNN
 F 3 "~" H 5150 4450 50  0001 C CNN
 	1    5150 4450
@@
 F 0 "C604" V 4750 4450 50  0000 L CNN
 F 1 "1uF" V 4850 4450 50  0000 L CNN
-F 2 "" H 4950 4600 50  0001 C CNN
+F 2 "Capacitor_SMD:C_0603_1608Metric_Pad1.05x0.95mm_HandSolder" H 4950 4600 50  0001 C CNN
 F 3 "~" H 4950 4600 50  0001 C CNN
 	1    4950 4600
@@
 F 0 "C606" V 5050 4650 50  0000 L CNN
 F 1 "1uF" V 5150 4650 50  0000 L CNN
-F 2 "" H 5250 4750 50  0001 C CNN
+F 2 "Capacitor_SMD:C_0603_1608Metric_Pad1.05x0.95mm_HandSolder" H 5250 4750 50  0001 C CNN
 F 3 "~" H 5250 4750 50  0001 C CNN
 	1    5250 4750
@@
 F 0 "C607" H 5750 4950 50  0000 L CNN
 F 1 "100nF" H 5700 5050 50  0000 L CNN
-F 2 "" H 5850 5150 50  0001 C CNN
+F 2 "Capacitor_SMD:C_0603_1608Metric_Pad1.05x0.95mm_HandSolder" H 5850 5150 50  0001 C CNN
 F 3 "~" H 5850 5150 50  0001 C CNN
 	1    5850 5150
@@
 F 0 "C608" H 5950 4950 50  0000 L CNN
 F 1 "100nF" H 5900 5050 50  0000 L CNN
-F 2 "" H 6050 5150 50  0001 C CNN
+F 2 "Capacitor_SMD:C_0603_1608Metric_Pad1.05x0.95mm_HandSolder" H 6050 5150 50  0001 C CNN
 F 3 "~" H 6050 5150 50  0001 C CNN
 	1    6050 5150
@@
 F 0 "C609" H 6150 4950 50  0000 L CNN
 F 1 "100nF" H 6100 5050 50  0000 L CNN
-F 2 "" H 6250 5150 50  0001 C CNN
+F 2 "Capacitor_SMD:C_0603_1608Metric_Pad1.05x0.95mm_HandSolder" H 6250 5150 50  0001 C CNN
 F 3 "~" H 6250 5150 50  0001 C CNN
 	1    6250 5150
@@
 F 0 "C610" H 6350 4950 50  0000 L CNN
 F 1 "100nF" H 6300 5050 50  0000 L CNN
-F 2 "" H 6450 5150 50  0001 C CNN
+F 2 "Capacitor_SMD:C_0603_1608Metric_Pad1.05x0.95mm_HandSolder" H 6450 5150 50  0001 C CNN
 F 3 "~" H 6450 5150 50  0001 C CNN
 	1    6450 5150
@@
 F 0 "C611" H 6550 5450 50  0000 L CNN
 F 1 "100nF" H 6500 5550 50  0000 L CNN
-F 2 "" H 6650 5650 50  0001 C CNN
+F 2 "Capacitor_SMD:C_0603_1608Metric_Pad1.05x0.95mm_HandSolder" H 6650 5650 50  0001 C CNN
 F 3 "~" H 6650 5650 50  0001 C CNN
 	1    6650 5650
@@
 F 0 "U601" H 4075 2665 50  0000 C CNN
 F 1 "XC6216C" H 4075 2574 50  0000 C CNN
-F 2 "" H 4100 2200 50  0001 C CNN
+F 2 "Package_TO_SOT_SMD:SOT-23-5_HandSoldering" H 4100 2200 50  0001 C CNN
 F 3 "/home/niko/kicad/datasheet/XC6216-XE6216.pdf" H 4100 2200 50  0001 C CNN
 	1    4100 2200
@@
 F 0 "R602" H 4609 2196 50  0000 L CNN
 F 1 "32K5" H 4609 2105 50  0000 L CNN
-F 2 "" H 4550 2150 50  0001 C CNN
+F 2 "Resistor_SMD:R_0603_1608Metric_Pad1.05x0.95mm_HandSolder" H 4550 2150 50  0001 C CNN
 F 3 "~" H 4550 2150 50  0001 C CNN
 	1    4550 2150
@@
 F 0 "R603" H 4609 2496 50  0000 L CNN
 F 1 "10K" H 4609 2405 50  0000 L CNN
-F 2 "" H 4550 2450 50  0001 C CNN
+F 2 "Resistor_SMD:R_0603_1608Metric_Pad1.05x0.95mm_HandSolder" H 4550 2450 50  0001 C CNN
 F 3 "~" H 4550 2450 50  0001 C CNN
 	1    4550 2450
@@
 F 0 "R601" H 3559 2496 50  0000 L CNN
 F 1 "10K" H 3559 2405 50  0000 L CNN
-F 2 "" H 3500 2450 50  0001 C CNN
+F 2 "Resistor_SMD:R_0603_1608Metric_Pad1.05x0.95mm_HandSolder" H 3500 2450 50  0001 C CNN
 F 3 "~" H 3500 2450 50  0001 C CNN
 	1    3500 2450
@@
 F 0 "C601" H 2250 2250 50  0000 L CNN
 F 1 "1uF" H 2200 2350 50  0000 L CNN
-F 2 "" H 2450 2350 50  0001 C CNN
+F 2 "Capacitor_SMD:C_0603_1608Metric_Pad1.05x0.95mm_HandSolder" H 2450 2350 50  0001 C CNN
 F 3 "~" H 2450 2350 50  0001 C CNN
 	1    2450 2350
@@
 F 0 "C602" H 4700 2250 50  0000 L CNN
 F 1 "1uF" H 4650 2350 50  0000 L CNN
-F 2 "" H 4900 2350 50  0001 C CNN
+F 2 "Capacitor_SMD:C_0603_1608Metric_Pad1.05x0.95mm_HandSolder" H 4900 2350 50  0001 C CNN
 F 3 "~" H 4900 2350 50  0001 C CNN
 	1    4900 2350
@@
 F 0 "R604" V 5550 4150 50  0000 C CNN
 F 1 "100R" V 5550 4450 50  0000 C CNN
-F 2 "" H 5650 4300 50  0001 C CNN
+F 2 "Resistor_SMD:R_0603_1608Metric_Pad1.05x0.95mm_HandSolder" H 5650 4300 50  0001 C CNN
 F 3 "~" H 5650 4300 50  0001 C CNN
 	1    5650 4300
@@
 F 0 "R605" V 5550 4300 50  0000 C CNN
 F 1 "100R" V 5550 4600 50  0000 C CNN
-F 2 "" H 5650 4450 50  0001 C CNN
+F 2 "Resistor_SMD:R_0603_1608Metric_Pad1.05x0.95mm_HandSolder" H 5650 4450 50  0001 C CNN
 F 3 "~" H 5650 4450 50  0001 C CNN
 	1    5650 4450
@@
 F 0 "R606" V 5550 4450 50  0000 C CNN
 F 1 "100R" V 5550 4750 50  0000 C CNN
-F 2 "" H 5650 4600 50  0001 C CNN
+F 2 "Resistor_SMD:R_0603_1608Metric_Pad1.05x0.95mm_HandSolder" H 5650 4600 50  0001 C CNN
 F 3 "~" H 5650 4600 50  0001 C CNN
 	1    5650 4600
@@
 F 0 "R607" V 5550 4600 50  0000 C CNN
 F 1 "100R" V 5550 4900 50  0000 C CNN
-F 2 "" H 5650 4750 50  0001 C CNN
+F 2 "Resistor_SMD:R_0603_1608Metric_Pad1.05x0.95mm_HandSolder" H 5650 4750 50  0001 C CNN
 F 3 "~" H 5650 4750 50  0001 C CNN
 	1    5650 4750
@@
 F 0 "R608" V 6350 3750 50  0000 C CNN
 F 1 "47R" V 6350 4050 50  0000 C CNN
-F 2 "" H 6450 3900 50  0001 C CNN
+F 2 "Resistor_SMD:R_0603_1608Metric_Pad1.05x0.95mm_HandSolder" H 6450 3900 50  0001 C CNN
 F 3 "~" H 6450 3900 50  0001 C CNN
 	1    6450 3900
@@
 F 0 "R609" V 6350 3900 50  0000 C CNN
 F 1 "47R" V 6350 4200 50  0000 C CNN
-F 2 "" H 6450 4050 50  0001 C CNN
+F 2 "Resistor_SMD:R_0603_1608Metric_Pad1.05x0.95mm_HandSolder" H 6450 4050 50  0001 C CNN
 F 3 "~" H 6450 4050 50  0001 C CNN
 	1    6450 4050
@@
 Wire Wire Line
 	6800 4050 6550 4050
-$Comp
-L Connector:AudioJack3_Ground J601
-U 1 1 5E85FCC9
-P 3050 4750
-F 0 "J601" H 3030 5075 50  0000 C CNN
-F 1 "AudioJack3_Ground" H 3030 4984 50  0000 C CNN
-F 2 "" H 3050 4750 50  0001 C CNN
-F 3 "~" H 3050 4750 50  0001 C CNN
-	1    3050 4750
-	1    0    0    -1
-$EndComp
-Text GLabel 3500 4850 2    50   Output ~ 0
-AUX_DETECT
-Wire Wire Line
-	3050 5200 3050 5050
+Wire Wire Line
+	3050 5200 3050 4950
 $Comp
 L power:GNDA #PWR0604
@@
 	7450 5750 7450 5500
 $Comp
-L Device:R_Small R610
-U 1 1 5EB72225
-P 3400 5100
-F 0 "R610" H 3459 5146 50  0000 L CNN
-F 1 "47K" H 3459 5055 50  0000 L CNN
-F 2 "" H 3400 5100 50  0001 C CNN
-F 3 "~" H 3400 5100 50  0001 C CNN
-	1    3400 5100
-	1    0    0    -1
-$EndComp
-Wire Wire Line
-	3400 5000 3400 4850
-Wire Wire Line
-	3250 4850 3400 4850
-$Comp
-L power:+3V3 #PWR0602
-U 1 1 5EB74D00
-P 3400 5200
-F 0 "#PWR0602" H 3400 5050 50  0001 C CNN
-F 1 "+3V3" H 3415 5373 50  0000 C CNN
-F 2 "" H 3400 5200 50  0001 C CNN
-F 3 "" H 3400 5200 50  0001 C CNN
-	1    3400 5200
-	-1   0    0    1
-$EndComp
-$Comp
 L Device:R_Small R611
 U 1 1 5EB80BE5
@@
 F 0 "R611" H 8509 4196 50  0000 L CNN
 F 1 "47K" H 8509 4105 50  0000 L CNN
-F 2 "" H 8450 4150 50  0001 C CNN
+F 2 "Resistor_SMD:R_0603_1608Metric_Pad1.05x0.95mm_HandSolder" H 8450 4150 50  0001 C CNN
 F 3 "~" H 8450 4150 50  0001 C CNN
 	1    8450 4150
@@
 F 0 "R612" H 8859 4196 50  0000 L CNN
 F 1 "DNP" H 8859 4105 50  0000 L CNN
-F 2 "" H 8800 4150 50  0001 C CNN
+F 2 "Resistor_SMD:R_0603_1608Metric_Pad1.05x0.95mm_HandSolder" H 8800 4150 50  0001 C CNN
 F 3 "~" H 8800 4150 50  0001 C CNN
 	1    8800 4150
@@
 $EndComp
 Wire Wire Line
-	3500 4850 3400 4850
-Connection ~ 3400 4850
-Wire Wire Line
 	4750 4600 4750 4650
 Wire Wire Line
@@
 F 0 "J602" H 5550 2217 50  0000 C CNN
 F 1 "Conn_02x01" H 5550 2126 50  0000 C CNN
-F 2 "" H 5500 2000 50  0001 C CNN
+F 2 "Connector_PinHeader_2.54mm:PinHeader_1x02_P2.54mm_Vertical" H 5500 2000 50  0001 C CNN
 F 3 "~" H 5500 2000 50  0001 C CNN
 	1    5500 2000
@@
 	6400 2000 6050 2000
 Connection ~ 6050 2000
+$Comp
+L Connector:AudioJack2_Ground J601
+U 1 1 5E98AE8D
+P 3050 4750
+F 0 "J601" H 3080 5075 50  0000 C CNN
+F 1 "SJ1-3533 CUI Devices" H 3080 4984 50  0000 C CNN
+F 2 "Connector_Audio:Jack_3.5mm_CUI_SJ1-3533NG_Horizontal" H 3050 4750 50  0001 C CNN
+F 3 "~" H 3050 4750 50  0001 C CNN
+	1    3050 4750
+	1    0    0    -1
+$EndComp
 $EndSCHEMATC

Commit message: PCB angefangen: Charger geplaced
Parts:
- removed J601: SJ1-3533 CUI Devices, Connector_Audio:Jack_3.5mm_CUI_SJ1-3533NG_Horizontal, symbol Connector:AudioJack2_Ground
- added J601: Conn_01x03_Female, Connector_PinHeader_2.54mm:PinHeader_1x03_P2.54mm_Vertical, symbol Connector:Conn_01x03_Female
- U602: footprint Package_SO:SOIC-18W_7.5x11.6mm_P1.27mm -> Package_SO:SOIC-20W_7.5x12.8mm_P1.27mm
Connections:
- net AUX_L: now also J601.3 (Pin_3)
- net AUX_R: now also J601.2 (Pin_2)
- net GNDA: now also J601.1 (Pin_1)
Changed lines of the file:
@@
 F 0 "U602" H 7450 4850 50  0000 C CNN
 F 1 "TDA7418" H 7450 4500 50  0000 C CNN
-F 2 "Package_SO:SOIC-18W_7.5x11.6mm_P1.27mm" H 7250 4700 50  0001 C CNN
+F 2 "Package_SO:SOIC-20W_7.5x12.8mm_P1.27mm" H 7250 4700 50  0001 C CNN
 F 3 "" H 7250 4700 50  0001 C CNN
 	1    7450 4650
@@
 Wire Wire Line
 	6800 4050 6550 4050
-Wire Wire Line
-	3050 5200 3050 4950
 $Comp
 L power:GNDA #PWR0604
@@
 Wire Wire Line
 	4750 4600 4750 4650
-Wire Wire Line
-	3250 4650 4750 4650
-Wire Wire Line
-	3250 4750 5150 4750
 Text Label 3750 4650 0    50   ~ 0
 AUX_L
@@
 Connection ~ 6050 2000
 $Comp
-L Connector:AudioJack2_Ground J601
-U 1 1 5E98AE8D
-P 3050 4750
-F 0 "J601" H 3080 5075 50  0000 C CNN
-F 1 "SJ1-3533 CUI Devices" H 3080 4984 50  0000 C CNN
-F 2 "Connector_Audio:Jack_3.5mm_CUI_SJ1-3533NG_Horizontal" H 3050 4750 50  0001 C CNN
-F 3 "~" H 3050 4750 50  0001 C CNN
-	1    3050 4750
-	1    0    0    -1
-$EndComp
+L Connector:Conn_01x03_Female J601
+U 1 1 5E973DDA
+P 2750 4750
+F 0 "J601" H 2644 4425 50  0000 C CNN
+F 1 "Conn_01x03_Female" H 2644 4516 50  0000 C CNN
+F 2 "Connector_PinHeader_2.54mm:PinHeader_1x03_P2.54mm_Vertical" H 2750 4750 50  0001 C CNN
+F 3 "~" H 2750 4750 50  0001 C CNN
+	1    2750 4750
+	-1   0    0    1
+$EndComp
+Wire Wire Line
+	2950 4650 4750 4650
+Wire Wire Line
+	2950 4750 5150 4750
+Wire Wire Line
+	2950 4850 3050 4850
+Wire Wire Line
+	3050 4850 3050 5200
 $EndSCHEMATC

Commit message: fertig zum routen
Parts:
- J601: footprint Connector_PinHeader_2.54mm:PinHeader_1x03_P2.54mm_Vertical -> Connector_PinHeader_2.54mm:PinHeader_1x03_P2.54mm_Vertical_SMD_Pin1Left
- J602: footprint Connector_PinHeader_2.54mm:PinHeader_1x02_P2.54mm_Vertical -> Connector_PinHeader_2.54mm:PinHeader_1x02_P2.54mm_Vertical_SMD_Pin1Left
Other:
- note added: "Audio DSP"
Changed lines of the file:
@@
 F 0 "J602" H 5550 2217 50  0000 C CNN
 F 1 "Conn_02x01" H 5550 2126 50  0000 C CNN
-F 2 "Connector_PinHeader_2.54mm:PinHeader_1x02_P2.54mm_Vertical" H 5500 2000 50  0001 C CNN
+F 2 "Connector_PinHeader_2.54mm:PinHeader_1x02_P2.54mm_Vertical_SMD_Pin1Left" H 5500 2000 50  0001 C CNN
 F 3 "~" H 5500 2000 50  0001 C CNN
 	1    5500 2000
@@
 F 0 "J601" H 2644 4425 50  0000 C CNN
 F 1 "Conn_01x03_Female" H 2644 4516 50  0000 C CNN
-F 2 "Connector_PinHeader_2.54mm:PinHeader_1x03_P2.54mm_Vertical" H 2750 4750 50  0001 C CNN
+F 2 "Connector_PinHeader_2.54mm:PinHeader_1x03_P2.54mm_Vertical_SMD_Pin1Left" H 2750 4750 50  0001 C CNN
 F 3 "~" H 2750 4750 50  0001 C CNN
 	1    2750 4750
@@
 Wire Wire Line
 	3050 4850 3050 5200
+Text Notes 6950 2750 0    128  ~ 0
+Audio DSP
 $EndSCHEMATC
