File: AudioProcessor.sch (KiCad schematic (older format))
At the start: 27 parts, among them J601 Conn_01x03_Female, J602 Conn_02x01, U601 XC6216C, U602 TDA7418

Commit message: Folienkondensatoren SMD gegen THT ausgetauscht. Kleine Fehler korrigiert
Parts:
- added C613: 1uF, Capacitor_THT:C_Rect_L7.0mm_W2.5mm_P5.00mm, symbol Device:C_Small
- added R610, R613, R614: 47K, Resistor_SMD:R_0603_1608Metric_Pad1.05x0.95mm_HandSolder, symbol Device:R_Small
- C603, C604, C605, C606, C607, C608, C609, C610: footprint Capacitor_SMD:C_0603_1608Metric_Pad1.05x0.95mm_HandSolder -> Capacitor_THT:C_Rect_L7.0mm_W2.5mm_P5.00mm
- C611: value 100nF -> 100nF 5%; footprint Capacitor_SMD:C_0603_1608Metric_Pad1.05x0.95mm_HandSolder -> Capacitor_THT:C_Rect_L7.0mm_W2.5mm_P5.00mm
Connections:
- wire segments 67 -> 70
- no-connect marks 6 -> 5
Other:
- moved on the sheet: C604, C606, C607, C608, C609, C610, J601, R606, R607

Commit message: layout fast fertig
Parts:
- added C614, C615, C616: 1uF, Capacitor_THT:C_Rect_L7.0mm_W2.5mm_P5.00mm, symbol Device:C_Small
- added J603: Conn_02x05_Odd_Even, Connector_PinHeader_2.54mm:PinHeader_2x05_P2.54mm_Vertical_SMD, symbol Connector_Generic:Conn_02x05_Odd_Even
- added R615, R616, R618, R619, R620: 1K, Resistor_SMD:R_0603_1608Metric_Pad1.05x0.95mm_HandSolder, symbol Device:R_Small
- added R617: 100K, Resistor_SMD:R_0603_1608Metric_Pad1.05x0.95mm_HandSolder, symbol Device:R_Small
Connections:
- wire segments 70 -> 106
- no-connect marks 5 -> 4
Other:
- moved on the sheet: J601

Commit message: Board abgeschickt
Parts:
- C603, C604, C605, C606, C613, C614, C615, C616: value 1uF -> 100nF
Connections:
- wire segments 106 -> 108
Changed lines of the file:
@@
 P 4950 4300
 F 0 "C603" V 4700 4250 50  0000 L CNN
-F 1 "1uF" V 4800 4250 50  0000 L CNN
+F 1 "100nF" V 4800 4250 50  0000 L CNN
 F 2 "Capacitor_THT:C_Rect_L7.0mm_W2.5mm_P5.00mm" H 4950 4300 50  0001 C CNN
 F 3 "https://www.mouser.de/datasheet/2/212/KEM_F3101_R82-1103738.pdf" H 4950 4300 50  0001 C CNN
@@
 P 5150 4450
 F 0 "C605" V 4950 4300 50  0000 L CNN
-F 1 "1uF" V 5050 4300 50  0000 L CNN
+F 1 "100nF" V 5050 4300 50  0000 L CNN
 F 2 "Capacitor_THT:C_Rect_L7.0mm_W2.5mm_P5.00mm" H 5150 4450 50  0001 C CNN
 F 3 "https://www.mouser.de/datasheet/2/212/KEM_F3101_R82-1103738.pdf" H 5150 4450 50  0001 C CNN
@@
 P 4750 4900
 F 0 "C604" V 4550 4750 50  0000 L CNN
-F 1 "1uF" V 4650 4750 50  0000 L CNN
+F 1 "100nF" V 4650 4750 50  0000 L CNN
 F 2 "Capacitor_THT:C_Rect_L7.0mm_W2.5mm_P5.00mm" H 4750 4900 50  0001 C CNN
 F 3 "https://www.mouser.de/datasheet/2/212/KEM_F3101_R82-1103738.pdf" H 4750 4900 50  0001 C CNN
@@
 P 5350 5200
 F 0 "C606" V 5150 5100 50  0000 L CNN
-F 1 "1uF" V 5250 5100 50  0000 L CNN
+F 1 "100nF" V 5250 5000 50  0000 L CNN
 F 2 "Capacitor_THT:C_Rect_L7.0mm_W2.5mm_P5.00mm" H 5350 5200 50  0001 C CNN
 F 3 "https://www.mouser.de/datasheet/2/212/KEM_F3101_R82-1103738.pdf" H 5350 5200 50  0001 C CNN
@@
 U 1 1 5E7DAB2A
 P 5650 5200
-F 0 "R607" V 5550 5050 50  0000 C CNN
-F 1 "100R" V 5550 5350 50  0000 C CNN
+F 0 "R607" V 5550 5150 50  0000 C CNN
+F 1 "100R" V 5550 5400 50  0000 C CNN
 F 2 "Resistor_SMD:R_0603_1608Metric_Pad1.05x0.95mm_HandSolder" H 5650 5200 50  0001 C CNN
 F 3 "~" H 5650 5200 50  0001 C CNN
@@
 Wire Wire Line
 	6800 3900 6550 3900
-Wire Wire Line
-	6800 4050 6550 4050
 $Comp
 L power:GNDA #PWR0604
@@
 P 5050 5050
 F 0 "C613" V 4850 4950 50  0000 L CNN
-F 1 "1uF" V 4950 4950 50  0000 L CNN
+F 1 "100nF" V 4950 4950 50  0000 L CNN
 F 2 "Capacitor_THT:C_Rect_L7.0mm_W2.5mm_P5.00mm" H 5050 5050 50  0001 C CNN
 F 3 "https://www.mouser.de/datasheet/2/212/KEM_F3101_R82-1103738.pdf" H 5050 5050 50  0001 C CNN
@@
 P 9050 4700
 F 0 "J603" H 9100 4350 50  0000 C CNN
-F 1 "Conn_02x05_Odd_Even" H 9100 4200 50  0000 C CNN
+F 1 "Conn_02x05_Odd_Even" H 9250 4150 50  0000 C CNN
 F 2 "Connector_PinHeader_2.54mm:PinHeader_2x05_P2.54mm_Vertical_SMD" H 9050 4700 50  0001 C CNN
 F 3 "~" H 9050 4700 50  0001 C CNN
@@
 AR Path="/5E751A81/5E9E91E1" Ref="C?"  Part="1"
 AR Path="/5EA6895E/5E9E91E1" Ref="C614"  Part="1"
-F 0 "C614" V 8300 4350 50  0000 C CNN
-F 1 "1uF" V 8300 4500 50  0000 C CNN
+F 0 "C614" V 8400 4250 50  0000 C CNN
+F 1 "100nF" V 8300 4250 50  0000 C CNN
 F 2 "Capacitor_THT:C_Rect_L7.0mm_W2.5mm_P5.00mm" H 8450 4400 50  0001 C CNN
 F 3 "~" H 8450 4400 50  0001 C CNN
@@
 AR Path="/5E751A81/5E9EBBE9" Ref="C?"  Part="1"
 AR Path="/5EA6895E/5E9EBBE9" Ref="C615"  Part="1"
-F 0 "C615" V 8550 4800 50  0000 C CNN
-F 1 "1uF" V 8550 4950 50  0000 C CNN
+F 0 "C615" V 8500 4700 50  0000 C CNN
+F 1 "100nF" V 8600 4700 50  0000 C CNN
 F 2 "Capacitor_THT:C_Rect_L7.0mm_W2.5mm_P5.00mm" H 8450 4850 50  0001 C CNN
 F 3 "~" H 8450 4850 50  0001 C CNN
@@
 AR Path="/5E751A81/5E9EBC75" Ref="C?"  Part="1"
 AR Path="/5EA6895E/5E9EBC75" Ref="C616"  Part="1"
-F 0 "C616" V 8300 4900 50  0000 C CNN
-F 1 "1uF" V 8300 5100 50  0000 C CNN
+F 0 "C616" V 8400 4850 50  0000 C CNN
+F 1 "100nF" V 8300 4850 50  0000 C CNN
 F 2 "Capacitor_THT:C_Rect_L7.0mm_W2.5mm_P5.00mm" H 8450 5000 50  0001 C CNN
 F 3 "~" H 8450 5000 50  0001 C CNN
@@
 	9750 4900 10000 4900
 Connection ~ 10000 4900
+Wire Wire Line
+	6800 4000 6650 4000
+Wire Wire Line
+	6650 4000 6650 4050
+Wire Wire Line
+	6650 4050 6550 4050
 $EndSCHEMATC

Commit message: mute and stdby tda7498 geändert, tda7418 durch tda7719 ersetzt, xs3868 durch bk8000l ersetzt, 3v3 stepdown statt LDO. BMS gelöscht.  TODO: Möglichkeit stepup und stepdown als modul aufzusetzen
Parts:
- removed C601, C602: 1uF, Capacitor_SMD:C_0603_1608Metric_Pad1.05x0.95mm_HandSolder, symbol Device:C_Small
- removed C607, C608, C614, C615, C616: 100nF, Capacitor_THT:C_Rect_L7.0mm_W2.5mm_P5.00mm, symbol Device:C_Small
- removed C611: 100nF 5%, Capacitor_THT:C_Rect_L7.0mm_W2.5mm_P5.00mm, symbol Device:C_Small
- removed J603: Conn_02x05_Odd_Even, Connector_PinHeader_2.54mm:PinHeader_2x05_P2.54mm_Vertical_SMD, symbol Connector_Generic:Conn_02x05_Odd_Even
- removed R602: 32K5, Resistor_SMD:R_0603_1608Metric_Pad1.05x0.95mm_HandSolder, symbol Device:R_Small
- removed R608, R609: 47R, Resistor_SMD:R_0603_1608Metric_Pad1.05x0.95mm_HandSolder, symbol Device:R_Small
- removed R611: 47K, Resistor_SMD:R_0603_1608Metric_Pad1.05x0.95mm_HandSolder, symbol Device:R_Small
- removed R612: DNP, Resistor_SMD:R_0603_1608Metric_Pad1.05x0.95mm_HandSolder, symbol Device:R_Small
- removed U602: TDA7418, Package_SO:SOIC-20W_7.5x12.8mm_P1.27mm, symbol MySymbols:TDA7418
- added C506, C508, C509, C536: 10u, Capacitor_THT:CP_Radial_D5.0mm_P2.50mm, symbol Device:CP1_Small
- added C537, C538, C539, C540: 1u, Capacitor_THT:C_Rect_L7.2mm_W7.2mm_P5.00mm_FKS2_FKP2_MKS2_MKP2, symbol Device:C_Small
- added J603: Conn_02x06_Odd_Even, symbol Connector_Generic:Conn_02x06_Odd_Even
- added Q501: 2N7002, Package_TO_SOT_SMD:SOT-23, symbol Transistor_FET:2N7002
- added R513, R515, R516, R517, R518: 10K, Resistor_SMD:R_0603_1608Metric_Pad1.05x0.95mm_HandSolder, symbol Device:R_Small
- added R514, R520, R521, R522, R523, R524: 100R, Resistor_SMD:R_0603_1608Metric_Pad1.05x0.95mm_HandSolder, symbol Device:R_Small
- added R519: 0R, Resistor_SMD:R_0603_1608Metric_Pad1.05x0.95mm_HandSolder, symbol Device:R_Small
- added R525: 1K, Resistor_SMD:R_0603_1608Metric_Pad1.05x0.95mm_HandSolder, symbol Device:R_Small
- added R526: DNP, Resistor_SMD:R_0603_1608Metric_Pad1.05x0.95mm_HandSolder, symbol Device:R_Small
- added TP501, TP502, TP503: TestPoint, TestPoint:TestPoint_Pad_2.0x2.0mm, symbol Connector:TestPoint
- added U502: BK8000L, symbol RF_Bluetooth:BK8000L
- added U503: TDA7719, Package_SO:TSSOP-28_4.4x9.7mm_P0.65mm, symbol MySymbols:TDA7719
- C603, C605: value 100nF -> 1u; footprint Capacitor_THT:C_Rect_L7.0mm_W2.5mm_P5.00mm -> Capacitor_THT:C_Rect_L7.2mm_W7.2mm_P5.00mm_FKS2_FKP2_MKS2_MKP2
- C604, C606, C609, C610, C613: value 100nF -> 1u
- J602: footprint Connector_PinHeader_2.54mm:PinHeader_1x02_P2.54mm_Vertical_SMD_Pin1Left -> Connector_PinHeader_2.54mm:PinHeader_1x02_P2.54mm_Vertical
- R610, R613, R614: value 47K -> 100K
- R617: value 100K -> DNP
Connections:
- net labels added: +3.3V, 8V5, BT_L+, BT_L-, BT_R+, BT_R-, RST_BT, RxT, TxR
- net labels removed: +3V3, +9V, BT_LEFT, BT_RIGHT, MUTE_TDA7418
- wire segments 108 -> 156
- no-connect marks 4 -> 20
Other:
- note added: "Bluetooth Module"
- note removed: "I2C Isolator?"
- moved on the sheet: C603, C604, C605, C606, C609, C610, C612, C613, J601, J602, R601, R603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

Commit message: neue schematic fertig zum rewiew. DRC clean
Parts:
- removed R520, R521, R522, R604, R605, R606, R607: 100R, Resistor_SMD:R_0603_1608Metric_Pad1.05x0.95mm_HandSolder, symbol Device:R_Small
- R523, R524: value 100R -> 47R
Connections:
- net AUX_L: no longer C604.2, J601.3 (Pin_3), R614.2
- net AUX_R: no longer C606.2, J601.1 (Pin_1), R610.2
- net BT_R+: now also C605.2; no longer C610.1
- net BT_R-: now also C610.1; no longer C605.2
- net at U503.10 (FDL+): now also C603.1
- net at U503.13 (FDR+): now also C605.1
- net at U503.1 (GD1L): now also C604.1
- net at U503.3 (QD1G): now also C606.1
- net at C609.2: now also U503.11 (FDL-)
- net at C610.2: now also U503.12 (FDR-)
- net at C613.1: now also U503.2 (GD1R)
- net 8V5 renamed +8V
- net ENABLE_9V renamed ENABLE_8V
- new net: C606.2, J601.1 (Pin_1), R610.2
- new net: C604.2, J601.3 (Pin_3), R614.2
- no-connect marks 20 -> 24
Other:
- moved on the sheet: C603, C604, C605, C606, C609, C610, C613, J601, R610, R613, R614

Commit message: module, falls schaltung nicht funktioniert hinzugefügt
Parts:
- added C541, C543, C544: 100nF, Capacitor_SMD:C_0603_1608Metric_Pad1.05x0.95mm_HandSolder, symbol Device:C_Small
- added C542: 10u, Capacitor_THT:CP_Radial_D5.0mm_P2.50mm, symbol Device:CP1_Small
- J603: footprint (none) -> Connector_PinHeader_2.54mm:PinHeader_2x06_P2.54mm_Vertical
- R519: footprint Resistor_SMD:R_0603_1608Metric_Pad1.05x0.95mm_HandSolder -> Resistor_SMD:R_1206_3216Metric_Pad1.42x1.75mm_HandSolder
- U502: footprint (none) -> RF_Module:BK8000L
Connections:
- net +3V3: now also C541.1, C542.1
- net +8V: now also C543.1, C544.1
- net GNDA: now also C541.2, C542.2, C543.2, C544.2
Changed lines of the file:
@@
 F 0 "J603" H 8500 4317 50  0000 C CNN
 F 1 "Conn_02x06_Odd_Even" H 8500 4226 50  0000 C CNN
-F 2 "" H 8450 3900 50  0001 C CNN
+F 2 "Connector_PinHeader_2.54mm:PinHeader_2x06_P2.54mm_Vertical" H 8450 3900 50  0001 C CNN
 F 3 "~" H 8450 3900 50  0001 C CNN
 	1    8450 3900
@@
 F 0 "U502" H 3525 7165 50  0000 C CNN
 F 1 "BK8000L" H 3525 7074 50  0000 C CNN
-F 2 "" H 3600 6250 50  0001 C CNN
+F 2 "RF_Module:BK8000L" H 3600 6250 50  0001 C CNN
 F 3 "/home/niko/kicad/datasheet/OVC3860-Datashett.pdf" H 3600 6250 50  0001 C CNN
 	1    3350 5800
@@
 Wire Wire Line
 	5400 3800 5400 3500
-Wire Wire Line
-	4550 5350 4100 5350
 Wire Wire Line
 	2950 5050 2700 5050
@@
 F 0 "R519" V 5000 1700 50  0000 C CNN
 F 1 "0R" V 5100 1700 50  0000 C CNN
-F 2 "Resistor_SMD:R_0603_1608Metric_Pad1.05x0.95mm_HandSolder" H 4850 1750 50  0001 C CNN
+F 2 "Resistor_SMD:R_1206_3216Metric_Pad1.42x1.75mm_HandSolder" H 4850 1750 50  0001 C CNN
 F 3 "~" H 4850 1750 50  0001 C CNN
 	1    4850 1750
@@
 L power:+8V #PWR0520
 U 1 1 5F316E62
-P 8250 3300
-F 0 "#PWR0520" H 8250 3150 50  0001 C CNN
-F 1 "+8V" H 8265 3473 50  0000 C CNN
-F 2 "" H 8250 3300 50  0001 C CNN
-F 3 "" H 8250 3300 50  0001 C CNN
-	1    8250 3300
+P 8250 2600
+F 0 "#PWR0520" H 8250 2450 50  0001 C CNN
+F 1 "+8V" H 8265 2773 50  0000 C CNN
+F 2 "" H 8250 2600 50  0001 C CNN
+F 3 "" H 8250 2600 50  0001 C CNN
+	1    8250 2600
 	1    0    0    -1
 $EndComp
@@
 NoConn ~ 2950 6350
 NoConn ~ 2950 6450
+$Comp
+L Device:C_Small C541
+U 1 1 5FE1C362
+P 5100 5500
+F 0 "C541" H 4750 5550 50  0000 L CNN
+F 1 "100nF" H 4700 5450 50  0000 L CNN
+F 2 "Capacitor_SMD:C_0603_1608Metric_Pad1.05x0.95mm_HandSolder" H 5100 5500 50  0001 C CNN
+F 3 "~" H 5100 5500 50  0001 C CNN
+	1    5100 5500
+	1    0    0    -1
+$EndComp
+$Comp
+L Device:CP1_Small C?
+U 1 1 5FE1C5A0
+P 5300 5500
+AR Path="/5E73BB4A/5FE1C5A0" Ref="C?"  Part="1"
+AR Path="/5EA6895E/5FE1C5A0" Ref="C542"  Part="1"
+F 0 "C542" H 5391 5546 50  0000 L CNN
+F 1 "10u" H 5391 5455 50  0000 L CNN
+F 2 "Capacitor_THT:CP_Radial_D5.0mm_P2.50mm" H 5300 5500 50  0001 C CNN
+F 3 "~" H 5300 5500 50  0001 C CNN
+	1    5300 5500
+	1    0    0    -1
+$EndComp
+Wire Wire Line
+	5300 5400 5300 5350
+Wire Wire Line
+	4100 5350 4550 5350
+Connection ~ 4550 5350
+Wire Wire Line
+	4550 5350 5100 5350
+Wire Wire Line
+	5100 5400 5100 5350
+Connection ~ 5100 5350
+Wire Wire Line
+	5100 5350 5300 5350
+$Comp
+L power:GNDA #PWR0521
+U 1 1 5FE36641
+P 5100 5750
+F 0 "#PWR0521" H 5100 5500 50  0001 C CNN
+F 1 "GNDA" H 5105 5577 50  0000 C CNN
+F 2 "" H 5100 5750 50  0001 C CNN
+F 3 "" H 5100 5750 50  0001 C CNN
+	1    5100 5750
+	1    0    0    -1
+$EndComp
+Wire Wire Line
+	5300 5700 5100 5700
+Wire Wire Line
+	5100 5700 5100 5750
+Wire Wire Line
+	5100 5600 5100 5700
+Connection ~ 5100 5700
+Wire Wire Line
+	5300 5600 5300 5700
+Wire Wire Line
+	8250 2600 8250 2650
+$Comp
+L Device:C_Small C543
+U 1 1 5FE53972
+P 8700 2850
+F 0 "C543" H 8350 2900 50  0000 L CNN
+F 1 "100nF" H 8300 2800 50  0000 L CNN
+F 2 "Capacitor_SMD:C_0603_1608Metric_Pad1.05x0.95mm_HandSolder" H 8700 2850 50  0001 C CNN
+F 3 "~" H 8700 2850 50  0001 C CNN
+	1    8700 2850
+	1    0    0    -1
+$EndComp
+$Comp
+L Device:C_Small C544
+U 1 1 5FE53AC9
+P 9200 2850
+F 0 "C544" H 8850 2900 50  0000 L CNN
+F 1 "100nF" H 8800 2800 50  0000 L CNN
+F 2 "Capacitor_SMD:C_0603_1608Metric_Pad1.05x0.95mm_HandSolder" H 9200 2850 50  0001 C CNN
+F 3 "~" H 9200 2850 50  0001 C CNN
+	1    9200 2850
+	1    0    0    -1
+$EndComp
+Wire Wire Line
+	9200 2750 9200 2650
+Wire Wire Line
+	9200 2650 8700 2650
+Connection ~ 8250 2650
+Wire Wire Line
+	8250 2650 8250 3300
+Wire Wire Line
+	8700 2750 8700 2650
+Connection ~ 8700 2650
+Wire Wire Line
+	8700 2650 8250 2650
+$Comp
+L power:GNDA #PWR0522
+U 1 1 5FE622C1
+P 8700 3000
+F 0 "#PWR0522" H 8700 2750 50  0001 C CNN
+F 1 "GNDA" H 8705 2827 50  0000 C CNN
+F 2 "" H 8700 3000 50  0001 C CNN
+F 3 "" H 8700 3000 50  0001 C CNN
+	1    8700 3000
+	1    0    0    -1
+$EndComp
+Wire Wire Line
+	9200 2950 8700 2950
+Wire Wire Line
+	8700 2950 8700 3000
+Connection ~ 8700 2950
 $EndSCHEMATC

Commit message: 3v3 regler ändern
Parts:
- C604, C606, C609, C610, C613: footprint Capacitor_THT:C_Rect_L7.0mm_W2.5mm_P5.00mm -> Capacitor_THT:C_Rect_L7.2mm_W7.2mm_P5.00mm_FKS2_FKP2_MKS2_MKP2
Changed lines of the file:
@@
 F 0 "C604" V 4700 2850 50  0000 L CNN
 F 1 "1u" V 4800 2850 50  0000 L CNN
-F 2 "Capacitor_THT:C_Rect_L7.0mm_W2.5mm_P5.00mm" H 4900 2800 50  0001 C CNN
+F 2 "Capacitor_THT:C_Rect_L7.2mm_W7.2mm_P5.00mm_FKS2_FKP2_MKS2_MKP2" H 4900 2800 50  0001 C CNN
 F 3 "https://www.mouser.de/datasheet/2/212/KEM_F3101_R82-1103738.pdf" H 4900 2800 50  0001 C CNN
 	1    4900 2800
@@
 F 0 "C606" V 4750 3250 50  0000 L CNN
 F 1 "1u" V 4850 3250 50  0000 L CNN
-F 2 "Capacitor_THT:C_Rect_L7.0mm_W2.5mm_P5.00mm" H 4900 3200 50  0001 C CNN
+F 2 "Capacitor_THT:C_Rect_L7.2mm_W7.2mm_P5.00mm_FKS2_FKP2_MKS2_MKP2" H 4900 3200 50  0001 C CNN
 F 3 "https://www.mouser.de/datasheet/2/212/KEM_F3101_R82-1103738.pdf" H 4900 3200 50  0001 C CNN
 	1    4900 3200
@@
 F 0 "C609" V 5250 3500 50  0000 L CNN
 F 1 "1u" V 5150 3550 50  0000 L CNN
-F 2 "Capacitor_THT:C_Rect_L7.0mm_W2.5mm_P5.00mm" H 5100 3700 50  0001 C CNN
+F 2 "Capacitor_THT:C_Rect_L7.2mm_W7.2mm_P5.00mm_FKS2_FKP2_MKS2_MKP2" H 5100 3700 50  0001 C CNN
 F 3 "https://www.mouser.de/datasheet/2/212/KEM_F3101_R82-1103738.pdf" H 5100 3700 50  0001 C CNN
 	1    5100 3700
@@
 F 0 "C610" V 5050 3900 50  0000 L CNN
 F 1 "1u" V 4950 3950 50  0000 L CNN
-F 2 "Capacitor_THT:C_Rect_L7.0mm_W2.5mm_P5.00mm" H 4900 3900 50  0001 C CNN
+F 2 "Capacitor_THT:C_Rect_L7.2mm_W7.2mm_P5.00mm_FKS2_FKP2_MKS2_MKP2" H 4900 3900 50  0001 C CNN
 F 3 "https://www.mouser.de/datasheet/2/212/KEM_F3101_R82-1103738.pdf" H 4900 3900 50  0001 C CNN
 	1    4900 3900
@@
 F 0 "C613" V 4750 3050 50  0000 L CNN
 F 1 "1u" V 4850 3050 50  0000 L CNN
-F 2 "Capacitor_THT:C_Rect_L7.0mm_W2.5mm_P5.00mm" H 4900 3000 50  0001 C CNN
+F 2 "Capacitor_THT:C_Rect_L7.2mm_W7.2mm_P5.00mm_FKS2_FKP2_MKS2_MKP2" H 4900 3000 50  0001 C CNN
 F 3 "https://www.mouser.de/datasheet/2/212/KEM_F3101_R82-1103738.pdf" H 4900 3000 50  0001 C CNN
 	1    4900 3000

Commit message: TODO: power on detect einfügen
Parts:
- TP501, TP502, TP503: footprint TestPoint:TestPoint_Pad_2.0x2.0mm -> TestPoint:TestPoint_Pad_1.0x1.0mm
Changed lines of the file:
@@
 F 0 "TP501" H 7258 2820 50  0000 L CNN
 F 1 "TestPoint" H 7258 2729 50  0000 L CNN
-F 2 "TestPoint:TestPoint_Pad_2.0x2.0mm" H 7400 2700 50  0001 C CNN
+F 2 "TestPoint:TestPoint_Pad_1.0x1.0mm" H 7400 2700 50  0001 C CNN
 F 3 "~" H 7400 2700 50  0001 C CNN
 	1    7200 2700
@@
 F 0 "TP502" H 7758 2820 50  0000 L CNN
 F 1 "TestPoint" H 7758 2729 50  0000 L CNN
-F 2 "TestPoint:TestPoint_Pad_2.0x2.0mm" H 7900 2700 50  0001 C CNN
+F 2 "TestPoint:TestPoint_Pad_1.0x1.0mm" H 7900 2700 50  0001 C CNN
 F 3 "~" H 7900 2700 50  0001 C CNN
 	1    7700 2700
@@
 F 0 "TP503" H 8458 3520 50  0000 L CNN
 F 1 "TestPoint" H 8458 3429 50  0000 L CNN
-F 2 "TestPoint:TestPoint_Pad_2.0x2.0mm" H 8600 3400 50  0001 C CNN
+F 2 "TestPoint:TestPoint_Pad_1.0x1.0mm" H 8600 3400 50  0001 C CNN
 F 3 "~" H 8600 3400 50  0001 C CNN
 	1    8400 3400
