File: AudioProcessor.sch (KiCad schematic (older format))
At the start: 68 parts, among them J601 Conn_01x03_Female, J602 Conn_02x01, J603 Conn_02x06_Odd_Even, Q501 2N7002, U502 BK8000L, U503 TDA7719, U504 AP2553AW6-7, U505 JW5026

Commit message: I2C Dreher behoben, BOM vereinfacht, 20dB Gain an ClassD Amps
Parts:
- C537: value 1u -> 1000p
- C604, C606, C613: value 1u -> 1u DNP
- J601: value Conn_01x03_Female -> DNP
- R523, R524: value 100R -> 47R
- R525, R615, R616, R619, R620: value 1K -> 0R
- R610: value 100R -> DNP
- R613, R614: value 100K -> DNP
- R618: value 1K -> OR
Connections:
- net SCL: now also R524.1; no longer R523.1
- net SDA: now also R523.1; no longer R524.1
Changed lines of the file:
@@
 EESchema Schematic File Version 4
-EELAYER 30 0
+LIBS:MukkeBox-cache
+EELAYER 26 0
 EELAYER END
 $Descr A4 11693 8268
@@
 Comment4 ""
 $EndDescr
-Text GLabel 7900 3200 2    50   BiDi ~ 0
+Text GLabel 7900 3050 2    50   BiDi ~ 0
 SDA
 Wire Wire Line
 	7550 3200 7900 3200
-Text GLabel 7900 3050 2    50   Input ~ 0
+Text GLabel 7900 3200 2    50   Input ~ 0
 SCL
 Wire Wire Line
@@
 P 4650 2900
 F 0 "C604" V 4550 2950 50  0000 L CNN
-F 1 "1u" V 4550 3200 50  0000 L CNN
+F 1 "1u DNP" V 4550 3200 50  0000 L CNN
 F 2 "Capacitor_THT:C_Rect_L7.2mm_W3.5mm_P5.00mm_FKS2_FKP2_MKS2_MKP2" H 4650 2900 50  0001 C CNN
 F 3 "https://www.mouser.de/datasheet/2/212/KEM_F3101_R82-1103738.pdf" H 4650 2900 50  0001 C CNN
@@
 P 4650 3100
 F 0 "C606" V 4600 3150 50  0000 L CNN
-F 1 "1u" V 4600 3350 50  0000 L CNN
+F 1 "1u DNP" V 4600 3350 50  0000 L CNN
 F 2 "Capacitor_THT:C_Rect_L7.2mm_W3.5mm_P5.00mm_FKS2_FKP2_MKS2_MKP2" H 4650 3100 50  0001 C CNN
 F 3 "https://www.mouser.de/datasheet/2/212/KEM_F3101_R82-1103738.pdf" H 4650 3100 50  0001 C CNN
@@
 P 3050 3000
 F 0 "J601" H 2944 2675 50  0000 C CNN
-F 1 "Conn_01x03_Female" H 2944 2766 50  0000 C CNN
+F 1 "DNP" H 2944 2766 50  0000 C CNN
 F 2 "Connector_PinHeader_2.54mm:PinHeader_1x03_P2.54mm_Vertical" H 3050 3000 50  0001 C CNN
 F 3 "~" H 3050 3000 50  0001 C CNN
@@
 P 3650 3350
 F 0 "R613" H 3500 3300 50  0000 C CNN
-F 1 "100K" H 3500 3400 50  0000 C CNN
+F 1 "DNP" H 3500 3400 50  0000 C CNN
 F 2 "Resistor_SMD:R_0603_1608Metric_Pad1.05x0.95mm_HandSolder" H 3650 3350 50  0001 C CNN
 F 3 "~" H 3650 3350 50  0001 C CNN
@@
 P 3950 3350
 F 0 "R614" H 3800 3300 50  0000 C CNN
-F 1 "100K" H 3800 3400 50  0000 C CNN
+F 1 "DNP" H 3800 3400 50  0000 C CNN
 F 2 "Resistor_SMD:R_0603_1608Metric_Pad1.05x0.95mm_HandSolder" H 3950 3350 50  0001 C CNN
 F 3 "~" H 3950 3350 50  0001 C CNN
@@
 P 5050 3000
 F 0 "C613" V 5000 3050 50  0000 L CNN
-F 1 "1u" V 5000 3300 50  0000 L CNN
+F 1 "1u DNP" V 5000 3300 50  0000 L CNN
 F 2 "Capacitor_THT:C_Rect_L7.2mm_W3.5mm_P5.00mm_FKS2_FKP2_MKS2_MKP2" H 5050 3000 50  0001 C CNN
 F 3 "https://www.mouser.de/datasheet/2/212/KEM_F3101_R82-1103738.pdf" H 5050 3000 50  0001 C CNN
@@
 P 3350 3350
 F 0 "R610" H 3200 3300 50  0000 C CNN
-F 1 "100R" H 3200 3400 50  0000 C CNN
+F 1 "DNP" H 3200 3400 50  0000 C CNN
 F 2 "Resistor_SMD:R_0603_1608Metric_Pad1.05x0.95mm_HandSolder" H 3350 3350 50  0001 C CNN
 F 3 "~" H 3350 3350 50  0001 C CNN
@@
 P 9050 3800
 F 0 "R615" V 9000 3900 50  0000 L CNN
-F 1 "1K" V 9000 3600 50  0000 L CNN
+F 1 "0R" V 9000 3600 50  0000 L CNN
 F 2 "Resistor_SMD:R_0603_1608Metric_Pad1.05x0.95mm_HandSolder" H 9050 3800 50  0001 C CNN
 F 3 "~" H 9050 3800 50  0001 C CNN
@@
 P 9050 3900
 F 0 "R616" V 9100 4000 50  0000 L CNN
-F 1 "1K" V 9000 3700 50  0000 L CNN
+F 1 "0R" V 9000 3700 50  0000 L CNN
 F 2 "Resistor_SMD:R_0603_1608Metric_Pad1.05x0.95mm_HandSolder" H 9050 3900 50  0001 C CNN
 F 3 "~" H 9050 3900 50  0001 C CNN
@@
 P 9050 4000
 F 0 "R619" V 9100 4100 50  0000 L CNN
-F 1 "1K" V 9000 3800 50  0000 L CNN
+F 1 "0R" V 9000 3800 50  0000 L CNN
 F 2 "Resistor_SMD:R_0603_1608Metric_Pad1.05x0.95mm_HandSolder" H 9050 4000 50  0001 C CNN
 F 3 "~" H 9050 4000 50  0001 C CNN
@@
 P 9050 4100
 F 0 "R620" V 9100 4200 50  0000 L CNN
-F 1 "1K" V 9000 3900 50  0000 L CNN
+F 1 "0R" V 9000 3900 50  0000 L CNN
 F 2 "Resistor_SMD:R_0603_1608Metric_Pad1.05x0.95mm_HandSolder" H 9050 4100 50  0001 C CNN
 F 3 "~" H 9050 4100 50  0001 C CNN
@@
 P 9050 3700
 F 0 "R618" V 9000 3800 50  0000 L CNN
-F 1 "1K" V 9000 3500 50  0000 L CNN
+F 1 "OR" V 9000 3500 50  0000 L CNN
 F 2 "Resistor_SMD:R_0603_1608Metric_Pad1.05x0.95mm_HandSolder" H 9050 3700 50  0001 C CNN
 F 3 "~" H 9050 3700 50  0001 C CNN
@@
 P 9050 4200
 F 0 "R525" V 9100 4300 50  0000 L CNN
-F 1 "1K" V 9000 4000 50  0000 L CNN
+F 1 "0R" V 9000 4000 50  0000 L CNN
 F 2 "Resistor_SMD:R_0603_1608Metric_Pad1.05x0.95mm_HandSolder" H 9050 4200 50  0001 C CNN
 F 3 "~" H 9050 4200 50  0001 C CNN
@@
 P 7450 3850
 F 0 "C537" V 7300 3900 50  0000 L CNN
-F 1 "1u" V 7400 3900 50  0000 L CNN
+F 1 "1000p" V 7400 3900 50  0000 L CNN
 F 2 "Capacitor_THT:C_Rect_L7.2mm_W3.5mm_P5.00mm_FKS2_FKP2_MKS2_MKP2" H 7450 3850 50  0001 C CNN
 F 3 "https://www.mouser.de/datasheet/2/212/KEM_F3101_R82-1103738.pdf" H 7450 3850 50  0001 C CNN
@@
 P 7450 3050
 F 0 "R523" V 7350 2900 50  0000 C CNN
-F 1 "100R" V 7350 3200 50  0000 C CNN
+F 1 "47R" V 7350 3200 50  0000 C CNN
 F 2 "Resistor_SMD:R_0603_1608Metric_Pad1.05x0.95mm_HandSolder" H 7450 3050 50  0001 C CNN
 F 3 "~" H 7450 3050 50  0001 C CNN
@@
 P 7450 3200
 F 0 "R524" V 7350 3050 50  0000 C CNN
-F 1 "100R" V 7350 3350 50  0000 C CNN
+F 1 "47R" V 7350 3350 50  0000 C CNN
 F 2 "Resistor_SMD:R_0603_1608Metric_Pad1.05x0.95mm_HandSolder" H 7450 3200 50  0001 C CNN
 F 3 "~" H 7450 3200 50  0001 C CNN
