File: 01_BMS.sch (KiCad schematic (older format))
At the start: 51 parts, among them J201 TB001-500-07BE CUI_Devices, Q201 NTD14N03RT4G, Q202 NTD14N03RT4G, Q203 NTD14N03RT4G, U201 BQ76920, U202 BQ76200

Commit message: Fertig zum letzten Check vor Bestellung
Parts:
- C212: footprint Capacitor_SMD:CP_Elec_6.3x5.9 -> Capacitor_THT:CP_Radial_D4.0mm_P2.00mm
Changed lines of the file:
@@
 F 0 "C212" H 5758 3004 50  0000 R CNN
 F 1 "4.7uF" H 5758 3095 50  0000 R CNN
-F 2 "Capacitor_SMD:CP_Elec_6.3x5.9" H 5850 3050 50  0001 C CNN
+F 2 "Capacitor_THT:CP_Radial_D4.0mm_P2.00mm" H 5850 3050 50  0001 C CNN
 F 3 "~" H 5850 3050 50  0001 C CNN
 	1    5850 3050

Commit message: Board abgeschickt
Parts:
- added R226: 10M, Resistor_SMD:R_0603_1608Metric_Pad1.05x0.95mm_HandSolder, symbol Device:R_Small
- C206, C207, C208: value 0.1uF -> 100nF
- R218: value xx -> 100K
- R219: value xx -> 10K
Connections:
- net CP_EN: now also R220.2
- net DISCHARGE_LOAD: now also R226.1
- net PACK+: now also R226.2
- net PCHG_EN: now also R224.2
- net PMON_EN: now also R222.2
- net at R221.2, U202.5 (CP_EN): no longer R220.2
- net at R223.2, U202.7 (PMON_EN): no longer R222.2
- net at R225.2, U202.8 (PCHG_EN): no longer R224.2
Other:
- moved on the sheet: R221, R223, R225
Changed lines of the file:
@@
 P 4150 4500
 F 0 "C207" V 3921 4500 50  0000 C CNN
-F 1 "0.1uF" V 4012 4500 50  0000 C CNN
+F 1 "100nF" V 4012 4500 50  0000 C CNN
 F 2 "Capacitor_SMD:C_0603_1608Metric_Pad1.05x0.95mm_HandSolder" H 4150 4500 50  0001 C CNN
 F 3 "~" H 4150 4500 50  0001 C CNN
@@
 P 3850 4500
 F 0 "C206" V 3621 4500 50  0000 C CNN
-F 1 "0.1uF" V 3712 4500 50  0000 C CNN
+F 1 "100nF" V 3712 4500 50  0000 C CNN
 F 2 "Capacitor_SMD:C_0603_1608Metric_Pad1.05x0.95mm_HandSolder" H 3850 4500 50  0001 C CNN
 F 3 "~" H 3850 4500 50  0001 C CNN
@@
 P 4450 4500
 F 0 "C208" V 4221 4500 50  0000 C CNN
-F 1 "0.1uF" V 4312 4500 50  0000 C CNN
+F 1 "100nF" V 4312 4500 50  0000 C CNN
 F 2 "Capacitor_SMD:C_0603_1608Metric_Pad1.05x0.95mm_HandSolder" H 4450 4500 50  0001 C CNN
 F 3 "~" H 4450 4500 50  0001 C CNN
@@
 	10200 1150 10200 2150
 Wire Wire Line
-	9850 1150 10100 1150
+	9850 1150 10000 1150
 Connection ~ 10200 2150
 Wire Wire Line
@@
 U 1 1 5E8D7080
 P 6150 2750
-F 0 "R217" V 6050 2700 50  0000 C CNN
-F 1 "10K" V 6050 2850 50  0000 C CNN
+F 0 "R217" V 5950 2750 50  0000 C CNN
+F 1 "10K" V 6050 2750 50  0000 C CNN
 F 2 "Resistor_SMD:R_0603_1608Metric_Pad1.05x0.95mm_HandSolder" H 6150 2750 50  0001 C CNN
 F 3 "~" H 6150 2750 50  0001 C CNN
@@
 L Device:R_Small R221
 U 1 1 5ED70E97
-P 9300 3700
-F 0 "R221" V 9250 3800 50  0000 C CNN
-F 1 "10K" V 9250 3550 50  0000 C CNN
-F 2 "Resistor_SMD:R_0603_1608Metric_Pad1.05x0.95mm_HandSolder" H 9300 3700 50  0001 C CNN
-F 3 "~" H 9300 3700 50  0001 C CNN
-	1    9300 3700
+P 9100 3700
+F 0 "R221" V 8900 3750 50  0000 C CNN
+F 1 "10K" V 9000 3750 50  0000 C CNN
+F 2 "Resistor_SMD:R_0603_1608Metric_Pad1.05x0.95mm_HandSolder" H 9100 3700 50  0001 C CNN
+F 3 "~" H 9100 3700 50  0001 C CNN
+	1    9100 3700
 	0    1    1    0
 $EndComp
@@
 L Device:R_Small R223
 U 1 1 5ED71182
-P 9550 3800
-F 0 "R223" V 9500 3900 50  0000 C CNN
-F 1 "10K" V 9500 3650 50  0000 C CNN
-F 2 "Resistor_SMD:R_0603_1608Metric_Pad1.05x0.95mm_HandSolder" H 9550 3800 50  0001 C CNN
-F 3 "~" H 9550 3800 50  0001 C CNN
-	1    9550 3800
+P 9350 3800
+F 0 "R223" V 9050 3850 50  0000 C CNN
+F 1 "10K" V 9150 3850 50  0000 C CNN
+F 2 "Resistor_SMD:R_0603_1608Metric_Pad1.05x0.95mm_HandSolder" H 9350 3800 50  0001 C CNN
+F 3 "~" H 9350 3800 50  0001 C CNN
+	1    9350 3800
 	0    1    1    0
 $EndComp
@@
 L Device:R_Small R225
 U 1 1 5ED711F0
-P 9800 3900
-F 0 "R225" V 9750 4000 50  0000 C CNN
-F 1 "10K" V 9750 3750 50  0000 C CNN
-F 2 "Resistor_SMD:R_0603_1608Metric_Pad1.05x0.95mm_HandSolder" H 9800 3900 50  0001 C CNN
-F 3 "~" H 9800 3900 50  0001 C CNN
-	1    9800 3900
+P 9600 3900
+F 0 "R225" V 9200 3950 50  0000 C CNN
+F 1 "10K" V 9300 3950 50  0000 C CNN
+F 2 "Resistor_SMD:R_0603_1608Metric_Pad1.05x0.95mm_HandSolder" H 9600 3900 50  0001 C CNN
+F 3 "~" H 9600 3900 50  0001 C CNN
+	1    9600 3900
 	0    1    1    0
 $EndComp
 Wire Wire Line
-	9400 3700 10050 3700
-Wire Wire Line
-	10050 3800 9650 3800
-Wire Wire Line
-	10050 3900 9900 3900
+	10050 3800 9450 3800
+Wire Wire Line
+	10050 3900 9700 3900
 $Comp
 L Device:R_Small R220
@@
 $EndComp
 Wire Wire Line
-	9700 4350 9700 3900
-Connection ~ 9700 3900
-Wire Wire Line
-	9700 3900 8900 3900
+	9500 3900 8900 3900
 $Comp
 L power:GND #PWR0202
@@
 $EndComp
 Wire Wire Line
-	9450 4350 9450 3800
-Connection ~ 9450 3800
-Wire Wire Line
-	8900 3800 9450 3800
-Wire Wire Line
-	9200 4350 9200 3700
-Connection ~ 9200 3700
-Wire Wire Line
-	8900 3700 9200 3700
+	8900 3800 9250 3800
+Wire Wire Line
+	8900 3700 9000 3700
 $Comp
 L Device:R_Small R218
 U 1 1 5EDF6B57
 P 8950 4450
-F 0 "R218" V 8850 4300 50  0000 R CNN
-F 1 "xx" V 8850 4550 50  0000 R CNN
+F 0 "R218" H 9200 4400 50  0000 R CNN
+F 1 "100K" H 9200 4500 50  0000 R CNN
 F 2 "Resistor_SMD:R_0603_1608Metric_Pad1.05x0.95mm_HandSolder" H 8950 4450 50  0001 C CNN
 F 3 "~" H 8950 4450 50  0001 C CNN
@@
 U 1 1 5EDF6BD1
 P 8950 5150
-F 0 "R219" V 8850 5000 50  0000 R CNN
-F 1 "xx" V 8850 5250 50  0000 R CNN
+F 0 "R219" H 9200 5100 50  0000 R CNN
+F 1 "10K" H 9200 5200 50  0000 R CNN
 F 2 "Resistor_SMD:R_0603_1608Metric_Pad1.05x0.95mm_HandSolder" H 8950 5150 50  0001 C CNN
 F 3 "~" H 8950 5150 50  0001 C CNN
@@
 F 1 "NTD14N03RT4G" V 9902 1250 50  0000 C CNN
 F 2 "Package_TO_SOT_SMD:TO-263-2" H 9850 1350 50  0001 C CNN
-F 3 "~" H 9650 1250 50  0001 C CNN
+F 3 "https://www.mouser.de/datasheet/2/308/NTD14N03R-D-1813942.pdf" H 9650 1250 50  0001 C CNN
 	1    9650 1250
 	0    1    -1   0
@@
 F 1 "NTD14N03RT4G" V 9400 2100 50  0000 C CNN
 F 2 "Package_TO_SOT_SMD:TO-263-2" H 9350 2350 50  0001 C CNN
-F 3 "~" H 9150 2250 50  0001 C CNN
+F 3 "https://www.mouser.de/datasheet/2/308/NTD14N03R-D-1813942.pdf" H 9150 2250 50  0001 C CNN
 	1    9150 2250
 	0    1    -1   0
@@
 F 1 "NTD14N03RT4G" V 9900 2100 50  0000 C CNN
 F 2 "Package_TO_SOT_SMD:TO-263-2" H 9850 2350 50  0001 C CNN
-F 3 "~" H 9650 2250 50  0001 C CNN
+F 3 "https://www.mouser.de/datasheet/2/308/NTD14N03R-D-1813942.pdf" H 9650 2250 50  0001 C CNN
 	1    9650 2250
 	0    -1   -1   0
@@
 	9350 1800 9350 2150
 Connection ~ 9350 2150
+$Comp
+L Device:R_Small R226
+U 1 1 5EAB52B8
+P 10000 1300
+F 0 "R226" V 10100 1300 50  0000 C CNN
+F 1 "10M" V 9900 1300 50  0000 C CNN
+F 2 "Resistor_SMD:R_0603_1608Metric_Pad1.05x0.95mm_HandSolder" H 10000 1300 50  0001 C CNN
+F 3 "~" H 10000 1300 50  0001 C CNN
+	1    10000 1300
+	-1   0    0    1
+$EndComp
+Wire Wire Line
+	10000 1200 10000 1150
+Connection ~ 10000 1150
+Wire Wire Line
+	10000 1150 10100 1150
+Wire Wire Line
+	10000 1400 10000 1450
+Wire Wire Line
+	10000 1450 9650 1450
+Connection ~ 9650 1450
+Wire Wire Line
+	9700 4350 9700 3900
+Connection ~ 9700 3900
+Wire Wire Line
+	9450 4350 9450 3800
+Connection ~ 9450 3800
+Wire Wire Line
+	9200 4350 9200 3700
+Connection ~ 9200 3700
+Wire Wire Line
+	9200 3700 10050 3700
 $EndSCHEMATC

Commit message: Letzter Kommit Version 0.1, Branch für neues Layout 0.2
Other:
- note added: "Charge Pump enable"
- note added: "Pack Monitor Enable"
- note added: "Precharge gate enable"
Changed lines of the file:
@@
 Wire Wire Line
 	9200 3700 10050 3700
+Text Notes 10550 3950 0    50   ~ 0
+Precharge gate enable
+Text Notes 10550 3850 0    50   ~ 0
+Pack Monitor Enable
+Text Notes 10550 3750 0    50   ~ 0
+Charge Pump enable
 $EndSCHEMATC
