File: Amplifier.sch (KiCad schematic (older format))
At the start: 58 parts, among them J501 TB001-500-04BE CUI_Devices, SW501 DS04-254-2-02BK-SMT, U501 TDA7498L

Commit message: neue schematic fertig zum rewiew. DRC clean
Parts:
- gave numbers to parts that had none: 6
Changed lines of the file:
@@
 L power:PWR_FLAG #FLG0111
 U 1 1 5EC21C56
-P 7700 3800
-F 0 "#FLG0111" H 7700 3875 50  0001 C CNN
-F 1 "PWR_FLAG" H 7700 3974 50  0000 C CNN
-F 2 "" H 7700 3800 50  0001 C CNN
-F 3 "~" H 7700 3800 50  0001 C CNN
-	1    7700 3800
+P 8400 3800
+F 0 "#FLG0111" H 8400 3875 50  0001 C CNN
+F 1 "PWR_FLAG" H 8400 3974 50  0000 C CNN
+F 2 "" H 8400 3800 50  0001 C CNN
+F 3 "~" H 8400 3800 50  0001 C CNN
+	1    8400 3800
 	1    0    0    -1
 $EndComp
@@
 	8800 3800 9050 3800
 Wire Wire Line
-	8250 3800 8550 3800
+	8250 3800 8400 3800
 Connection ~ 8250 3800
 Connection ~ 8550 3800
@@
 	4300 2250 4750 2250
 $Comp
-L power:GND #PWR?
+L power:GND #PWR0413
 U 1 1 5EEA9F5C
 P 6800 5700
-F 0 "#PWR?" H 6800 5450 50  0001 C CNN
+F 0 "#PWR0413" H 6800 5450 50  0001 C CNN
 F 1 "GND" H 6805 5527 50  0000 C CNN
 F 2 "" H 6800 5700 50  0001 C CNN
@@
 $EndComp
 $Comp
-L power:GND #PWR?
+L power:GND #PWR0412
 U 1 1 5EEAA0E6
 P 6350 5700
-F 0 "#PWR?" H 6350 5450 50  0001 C CNN
+F 0 "#PWR0412" H 6350 5450 50  0001 C CNN
 F 1 "GND" H 6355 5527 50  0000 C CNN
 F 2 "" H 6350 5700 50  0001 C CNN
@@
 $EndComp
 $Comp
-L power:GND #PWR?
+L power:GND #PWR0411
 U 1 1 5EEB6CAA
 P 4550 6450
-F 0 "#PWR?" H 4550 6200 50  0001 C CNN
+F 0 "#PWR0411" H 4550 6200 50  0001 C CNN
 F 1 "GND" H 4650 6350 50  0000 C CNN
 F 2 "" H 4550 6450 50  0001 C CNN
@@
 $EndComp
 $Comp
-L power:GND #PWR?
+L power:GND #PWR0410
 U 1 1 5EEB6EFD
 P 4000 6450
-F 0 "#PWR?" H 4000 6200 50  0001 C CNN
+F 0 "#PWR0410" H 4000 6200 50  0001 C CNN
 F 1 "GND" H 4100 6350 50  0000 C CNN
 F 2 "" H 4000 6450 50  0001 C CNN
@@
 $EndComp
 $Comp
-L power:GND #PWR?
+L power:GND #PWR0408
 U 1 1 5EEB7040
 P 3300 4250
-F 0 "#PWR?" H 3300 4000 50  0001 C CNN
+F 0 "#PWR0408" H 3300 4000 50  0001 C CNN
 F 1 "GND" H 3305 4077 50  0000 C CNN
 F 2 "" H 3300 4250 50  0001 C CNN
@@
 	3300 4250 3500 4250
 $Comp
-L power:GND #PWR?
+L power:GND #PWR0405
 U 1 1 5EEB7231
 P 3050 2750
-F 0 "#PWR?" H 3050 2500 50  0001 C CNN
+F 0 "#PWR0405" H 3050 2500 50  0001 C CNN
 F 1 "GND" H 3055 2577 50  0000 C CNN
 F 2 "" H 3050 2750 50  0001 C CNN
@@
 	3050 2750 3000 2750
 $Comp
-L power:GND #PWR?
+L power:GND #PWR0414
 U 1 1 5EEB78DA
 P 7700 3800
-F 0 "#PWR?" H 7700 3550 50  0001 C CNN
+F 0 "#PWR0414" H 7700 3550 50  0001 C CNN
 F 1 "GND" H 7705 3627 50  0000 C CNN
 F 2 "" H 7700 3800 50  0001 C CNN
@@
 Connection ~ 7700 3800
 $Comp
-L power:+3.3V #PWR?
+L power:+3.3V #PWR0401
 U 1 1 5EEBB7BD
 P 1750 5400
-F 0 "#PWR?" H 1750 5250 50  0001 C CNN
+F 0 "#PWR0401" H 1750 5250 50  0001 C CNN
 F 1 "+3.3V" H 1765 5573 50  0000 C CNN
 F 2 "" H 1750 5400 50  0001 C CNN
@@
 P 2650 6250
 AR Path="/5E73BB4A/5EF0C11E" Ref="Q?"  Part="1"
-AR Path="/5E751A81/5EF0C11E" Ref="Q?"  Part="1"
-F 0 "Q?" H 2850 6450 50  0000 L CNN
+AR Path="/5E751A81/5EF0C11E" Ref="Q401"  Part="1"
+F 0 "Q401" H 2850 6450 50  0000 L CNN
 F 1 "2N7002" H 2850 6350 50  0000 L CNN
 F 2 "Package_TO_SOT_SMD:SOT-23" H 2850 6175 50  0001 L CIN
@@
 P 3450 6850
 AR Path="/5E73BB4A/5EF1626F" Ref="Q?"  Part="1"
-AR Path="/5E751A81/5EF1626F" Ref="Q?"  Part="1"
-F 0 "Q?" H 3650 7050 50  0000 L CNN
+AR Path="/5E751A81/5EF1626F" Ref="Q402"  Part="1"
+F 0 "Q402" H 3650 7050 50  0000 L CNN
 F 1 "2N7002" H 3650 6950 50  0000 L CNN
 F 2 "Package_TO_SOT_SMD:SOT-23" H 3650 6775 50  0001 L CIN
@@
 	3550 5700 2500 5700
 $Comp
-L power:GND #PWR?
+L power:GND #PWR0403
 U 1 1 5EF3FD4E
 P 2750 6450
-F 0 "#PWR?" H 2750 6200 50  0001 C CNN
+F 0 "#PWR0403" H 2750 6200 50  0001 C CNN
 F 1 "GND" H 2850 6350 50  0000 C CNN
 F 2 "" H 2750 6450 50  0001 C CNN
@@
 $EndComp
 $Comp
-L power:GND #PWR?
+L power:GND #PWR0409
 U 1 1 5EF3FDC5
 P 3550 7050
-F 0 "#PWR?" H 3550 6800 50  0001 C CNN
+F 0 "#PWR0409" H 3550 6800 50  0001 C CNN
 F 1 "GND" H 3650 6950 50  0000 C CNN
 F 2 "" H 3550 7050 50  0001 C CNN
@@
 	4000 6100 4000 6450
 $Comp
-L Device:R_Small R?
+L Device:R_Small R411
 U 1 1 5EF6B464
 P 2250 6350
-F 0 "R?" H 2500 6300 50  0000 C CNN
+F 0 "R411" H 2500 6300 50  0000 C CNN
 F 1 "100K" H 2450 6400 50  0000 C CNN
 F 2 "Resistor_SMD:R_0603_1608Metric_Pad1.05x0.95mm_HandSolder" H 2250 6350 50  0001 C CNN
@@
 $EndComp
 $Comp
-L Device:R_Small R?
+L Device:R_Small R418
 U 1 1 5EF6B555
 P 3050 6950
-F 0 "R?" H 3250 6900 50  0000 C CNN
+F 0 "R418" H 3250 6900 50  0000 C CNN
 F 1 "100K" H 3200 7000 50  0000 C CNN
 F 2 "Resistor_SMD:R_0603_1608Metric_Pad1.05x0.95mm_HandSolder" H 3050 6950 50  0001 C CNN
@@
 Connection ~ 2750 6450
 $Comp
-L Device:R_Small R?
+L Device:R_Small R414
 U 1 1 5EF8E991
 P 2350 6250
-F 0 "R?" V 2154 6250 50  0000 C CNN
+F 0 "R414" V 2154 6250 50  0000 C CNN
 F 1 "1K" V 2245 6250 50  0000 C CNN
 F 2 "Resistor_SMD:R_0603_1608Metric_Pad1.05x0.95mm_HandSolder" H 2350 6250 50  0001 C CNN
@@
 $EndComp
 $Comp
-L Device:R_Small R?
+L Device:R_Small R419
 U 1 1 5EFB0278
 P 3150 6850
-F 0 "R?" V 2954 6850 50  0000 C CNN
+F 0 "R419" V 2954 6850 50  0000 C CNN
 F 1 "1K" V 3045 6850 50  0000 C CNN
 F 2 "Resistor_SMD:R_0603_1608Metric_Pad1.05x0.95mm_HandSolder" H 3150 6850 50  0001 C CNN
@@
 	1750 5700 2300 5700
 Connection ~ 1750 5550
+Connection ~ 8400 3800
+Wire Wire Line
+	8400 3800 8550 3800
 $EndSCHEMATC
