File: _saved_00_Charger.sch (KiCad schematic (older format))
At the start: 55 parts, among them J303 TB001-500-02BE CUI_Devices, J401 TB001-500-02BE CUI_Devices, Q303 2N7002, Q304 2N7002, Q305 FDD4685-F085, Q306 2N7002, Q307 BSS84, Q308 2N7002, Q309 FDD4685-F085, U401 MAX1873TEEE

Commit message: TODO: power on detect einfügen
Parts:
- added C301: 100n, Capacitor_SMD:C_0603_1608Metric_Pad1.05x0.95mm_HandSolder, symbol Device:C_Small
Connections:
- net CHARGER_IOUT: now also C301.1
- net GND: now also C301.2
Changed lines of the file:
@@
 	1    0    0    -1
 $EndComp
+$Comp
+L Device:C_Small C301
+U 1 1 5ED2EDE0
+P 2650 4300
+F 0 "C301" H 2800 4400 50  0000 C CNN
+F 1 "100n" H 2850 4300 50  0000 C CNN
+F 2 "Capacitor_SMD:C_0603_1608Metric_Pad1.05x0.95mm_HandSolder" H 2650 4300 50  0001 C CNN
+F 3 "~" H 2650 4300 50  0001 C CNN
+	1    2650 4300
+	1    0    0    -1
+$EndComp
+Wire Wire Line
+	2650 4200 2650 3950
+Wire Wire Line
+	2650 3950 2250 3950
+$Comp
+L power:GND #PWR0307
+U 1 1 5ED36D0B
+P 2650 4600
+F 0 "#PWR0307" H 2650 4350 50  0001 C CNN
+F 1 "GND" H 2655 4427 50  0000 C CNN
+F 2 "" H 2650 4600 50  0001 C CNN
+F 3 "" H 2650 4600 50  0001 C CNN
+	1    2650 4600
+	1    0    0    -1
+$EndComp
+Wire Wire Line
+	2650 4400 2650 4600
 $EndSCHEMATC
