File: 00_Charger.sch (KiCad schematic (older format))
At the start: 46 parts, among them J303 TB001-500-02BE CUI_Devices, J401 TB001-500-02BE CUI_Devices, Q303 2N7002, Q304 2N7002, Q305 FDD4685-F085, Q306 2N7002, Q402 FDD4685-F085, U401 MAX1873TEEE

Commit message: neue schematic fertig zum rewiew. DRC clean
Parts:
- removed Q402: FDD4685-F085, Package_TO_SOT_SMD:TO-252-2, symbol Device:Q_NMOS_GSD
- added C309: 100n, Capacitor_SMD:C_0603_1608Metric_Pad1.05x0.95mm_HandSolder, symbol Device:C_Small
- added Q307: BSS84, Package_TO_SOT_SMD:SOT-23, symbol Transistor_FET:BSS84
- added Q308: 2N7002, Package_TO_SOT_SMD:SOT-23, symbol Transistor_FET:2N7002
- added Q309: FDD4685-F085, Package_TO_SOT_SMD:TO-252-2, symbol Device:Q_PMOS_GDS
- added R313: 470K, Resistor_SMD:R_0603_1608Metric_Pad1.05x0.95mm_HandSolder, symbol Device:R_Small
- added R314: 47K, Resistor_SMD:R_0603_1608Metric_Pad1.05x0.95mm_HandSolder, symbol Device:R_Small
- added R315, R316, R318: 100K, Resistor_SMD:R_0603_1608Metric_Pad1.05x0.95mm_HandSolder, symbol Device:R_Small
- added R317: 1K, Resistor_SMD:R_0603_1608Metric_Pad1.05x0.95mm_HandSolder, symbol Device:R_Small
Connections:
- net GND: now also C309.2, Q308.2 (S), R314.1, R318.1
- net PACK+: now also Q307.2 (S), R315.2
- net at U401.14 (EXT): now also Q309.1 (G)
- net at C412.1, Q305.3 (D), R307.2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: now also Q309.3 (S)
- net at D402.2 (K), L302.1: now also Q309.2 (D)
- new net: Q307.1 (G), R315.1, R316.2
- new net: Q307.3 (D), R313.2
- new net: Q308.1 (G), R317.2
- new net: Q308.3 (D), R316.1
- new net EN_PACK_SENSE: R317.1, R318.2
- new net PACK_SENSE: C309.1, R313.1, R314.2
Other:
- note added: "1,64V bei 18V Eingangsspannung"
- moved on the sheet: F301, J303
Changed lines of the file:
@@
 	0    1    1    0
 $EndComp
-Text Notes 650  6450 0    50   ~ 0
+Text Notes 750  5550 0    50   ~ 0
 Zum Lition-Zellen-Block
 $Comp
@@
 	-1   0    0    1
 $EndComp
-$Comp
-L Device:Q_NMOS_GSD Q402
-U 1 1 5E98AB96
-P 7750 3550
-F 0 "Q402" H 7600 3350 50  0000 L CNN
-F 1 "FDD4685-F085" H 7200 3250 50  0000 L CNN
-F 2 "Package_TO_SOT_SMD:TO-252-2" H 7950 3650 50  0001 C CNN
-F 3 "https://www.mouser.de/datasheet/2/308/FDD4685_F085-D-1807000.pdf" H 7750 3550 50  0001 C CNN
-	1    7750 3550
-	1    0    0    -1
-$EndComp
-Connection ~ 7850 3750
-Connection ~ 7850 3350
 $Comp
 L Device:D_Schottky_x2_KCom_AKA D?
@@
 	1    0    0    -1
 $EndComp
-Text GLabel 2000 7050 2    50   BiDi ~ 0
+Text GLabel 2900 6150 2    50   BiDi ~ 0
 PACK+
 $Comp
 L Connector:Screw_Terminal_01x02 J303
 U 1 1 5ED37ADF
-P 1150 7150
-F 0 "J303" H 1400 6800 50  0000 C CNN
-F 1 "TB001-500-02BE CUI_Devices" V 1550 7150 50  0000 C CNN
-F 2 "TerminalBlock_RND:TerminalBlock_RND_205-00045_1x02_P5.00mm_Horizontal" H 1150 7150 50  0001 C CNN
-F 3 "https://www.mouser.de/datasheet/2/670/tb001-500-1550615.pdf" H 1150 7150 50  0001 C CNN
-	1    1150 7150
+P 1250 6250
+F 0 "J303" H 1500 5900 50  0000 C CNN
+F 1 "TB001-500-02BE CUI_Devices" V 1650 6250 50  0000 C CNN
+F 2 "TerminalBlock_RND:TerminalBlock_RND_205-00045_1x02_P5.00mm_Horizontal" H 1250 6250 50  0001 C CNN
+F 3 "https://www.mouser.de/datasheet/2/670/tb001-500-1550615.pdf" H 1250 6250 50  0001 C CNN
+	1    1250 6250
 	-1   0    0    1
 $EndComp
@@
 L power:GND #PWR0301
 U 1 1 5ED37D03
-P 1400 7250
-F 0 "#PWR0301" H 1400 7000 50  0001 C CNN
-F 1 "GND" H 1405 7077 50  0000 C CNN
-F 2 "" H 1400 7250 50  0001 C CNN
-F 3 "" H 1400 7250 50  0001 C CNN
-	1    1400 7250
-	1    0    0    -1
-$EndComp
-Wire Wire Line
-	1400 7150 1350 7150
-Wire Wire Line
-	1400 7150 1400 7250
+P 1500 6350
+F 0 "#PWR0301" H 1500 6100 50  0001 C CNN
+F 1 "GND" H 1505 6177 50  0000 C CNN
+F 2 "" H 1500 6350 50  0001 C CNN
+F 3 "" H 1500 6350 50  0001 C CNN
+	1    1500 6350
+	1    0    0    -1
+$EndComp
+Wire Wire Line
+	1500 6250 1450 6250
+Wire Wire Line
+	1500 6250 1500 6350
 Wire Wire Line
 	10600 3250 10500 3250
@@
 L Device:Fuse_Small F301
 U 1 1 5EDE4BFA
-P 1750 7050
-F 0 "F301" H 1750 7235 50  0000 C CNN
-F 1 "Fuse_Small" H 1750 7144 50  0000 C CNN
-F 2 "Fuse:Fuseholder_Cylinder-5x20mm_Schurter_0031-8002_Horizontal_Open" H 1750 7050 50  0001 C CNN
-F 3 "~" H 1750 7050 50  0001 C CNN
-	1    1750 7050
-	1    0    0    -1
-$EndComp
-Wire Wire Line
-	1350 7050 1650 7050
+P 1850 6150
+F 0 "F301" H 1850 6335 50  0000 C CNN
+F 1 "Fuse_Small" H 1850 6244 50  0000 C CNN
+F 2 "Fuse:Fuseholder_Cylinder-5x20mm_Schurter_0031-8002_Horizontal_Open" H 1850 6150 50  0001 C CNN
+F 3 "~" H 1850 6150 50  0001 C CNN
+	1    1850 6150
+	1    0    0    -1
+$EndComp
+Wire Wire Line
+	1450 6150 1750 6150
 Wire Wire Line
 	7850 3750 8450 3750
@@
 Wire Wire Line
 	2500 2200 3950 2200
-Wire Wire Line
-	1850 7050 2000 7050
 Text GLabel 10800 4450 2    50   Input ~ 0
 PWR_EN
@@
 Text Notes 4950 3850 0    50   ~ 0
 ca. 4-5V
+$Comp
+L Transistor_FET:BSS84 Q307
+U 1 1 5F19A986
+P 2400 6650
+F 0 "Q307" H 2606 6604 50  0000 L CNN
+F 1 "BSS84" H 2606 6695 50  0000 L CNN
+F 2 "Package_TO_SOT_SMD:SOT-23" H 2600 6575 50  0001 L CIN
+F 3 "http://assets.nexperia.com/documents/data-sheet/BSS84.pdf" H 2400 6650 50  0001 L CNN
+	1    2400 6650
+	-1   0    0    1
+$EndComp
+Wire Wire Line
+	2300 6450 2300 6150
+Wire Wire Line
+	1950 6150 2300 6150
+Wire Wire Line
+	2900 6150 2850 6150
+Connection ~ 2300 6150
+$Comp
+L Transistor_FET:2N7002 Q308
+U 1 1 5F1BD299
+P 2950 7300
+F 0 "Q308" H 3155 7346 50  0000 L CNN
+F 1 "2N7002" H 3155 7255 50  0000 L CNN
+F 2 "Package_TO_SOT_SMD:SOT-23" H 3150 7225 50  0001 L CIN
+F 3 "https://www.fairchildsemi.com/datasheets/2N/2N7002.pdf" H 2950 7300 50  0001 L CNN
+	1    2950 7300
+	-1   0    0    -1
+$EndComp
+$Comp
+L Device:R_Small R316
+U 1 1 5F1C25F3
+P 2850 6900
+F 0 "R316" H 2791 6854 50  0000 R CNN
+F 1 "100K" H 2791 6945 50  0000 R CNN
+F 2 "Resistor_SMD:R_0603_1608Metric_Pad1.05x0.95mm_HandSolder" H 2850 6900 50  0001 C CNN
+F 3 "~" H 2850 6900 50  0001 C CNN
+	1    2850 6900
+	-1   0    0    1
+$EndComp
+$Comp
+L Device:R_Small R315
+U 1 1 5F1C28BE
+P 2850 6400
+F 0 "R315" H 2791 6354 50  0000 R CNN
+F 1 "100K" H 2791 6445 50  0000 R CNN
+F 2 "Resistor_SMD:R_0603_1608Metric_Pad1.05x0.95mm_HandSolder" H 2850 6400 50  0001 C CNN
+F 3 "~" H 2850 6400 50  0001 C CNN
+	1    2850 6400
+	-1   0    0    1
+$EndComp
+Wire Wire Line
+	2850 6300 2850 6150
+Connection ~ 2850 6150
+Wire Wire Line
+	2850 6150 2300 6150
+Wire Wire Line
+	2850 6500 2850 6650
+Wire Wire Line
+	2850 6650 2600 6650
+Wire Wire Line
+	2850 6650 2850 6800
+Connection ~ 2850 6650
+Wire Wire Line
+	2850 7000 2850 7100
+$Comp
+L power:GND #PWR0306
+U 1 1 5F1D7D48
+P 2850 7550
+F 0 "#PWR0306" H 2850 7300 50  0001 C CNN
+F 1 "GND" H 2855 7377 50  0000 C CNN
+F 2 "" H 2850 7550 50  0001 C CNN
+F 3 "" H 2850 7550 50  0001 C CNN
+	1    2850 7550
+	1    0    0    -1
+$EndComp
+Wire Wire Line
+	2850 7550 2850 7500
+$Comp
+L Device:R_Small R318
+U 1 1 5F1DD6B9
+P 3450 7450
+F 0 "R318" H 3391 7404 50  0000 R CNN
+F 1 "100K" H 3391 7495 50  0000 R CNN
+F 2 "Resistor_SMD:R_0603_1608Metric_Pad1.05x0.95mm_HandSolder" H 3450 7450 50  0001 C CNN
+F 3 "~" H 3450 7450 50  0001 C CNN
+	1    3450 7450
+	-1   0    0    1
+$EndComp
+Wire Wire Line
+	3450 7550 2850 7550
+Connection ~ 2850 7550
+$Comp
+L Device:R_Small R317
+U 1 1 5F1E33A0
+P 3300 7300
+F 0 "R317" V 3100 7300 50  0000 C CNN
+F 1 "1K" V 3200 7300 50  0000 C CNN
+F 2 "Resistor_SMD:R_0603_1608Metric_Pad1.05x0.95mm_HandSolder" H 3300 7300 50  0001 C CNN
+F 3 "~" H 3300 7300 50  0001 C CNN
+	1    3300 7300
+	0    1    1    0
+$EndComp
+Wire Wire Line
+	3450 7350 3450 7300
+Wire Wire Line
+	3450 7300 3400 7300
+Wire Wire Line
+	3200 7300 3150 7300
+$Comp
+L Device:R_Small R313
+U 1 1 5F1F0273
+P 2300 7050
+F 0 "R313" H 2600 7000 50  0000 R CNN
+F 1 "470K" H 2600 7100 50  0000 R CNN
+F 2 "Resistor_SMD:R_0603_1608Metric_Pad1.05x0.95mm_HandSolder" H 2300 7050 50  0001 C CNN
+F 3 "~" H 2300 7050 50  0001 C CNN
+	1    2300 7050
+	-1   0    0    1
+$EndComp
+Wire Wire Line
+	2300 6950 2300 6850
+$Comp
+L Device:R_Small R314
+U 1 1 5F1F63D6
+P 2300 7350
+F 0 "R314" H 2600 7300 50  0000 R CNN
+F 1 "47K" H 2600 7400 50  0000 R CNN
+F 2 "Resistor_SMD:R_0603_1608Metric_Pad1.05x0.95mm_HandSolder" H 2300 7350 50  0001 C CNN
+F 3 "~" H 2300 7350 50  0001 C CNN
+	1    2300 7350
+	-1   0    0    1
+$EndComp
+Wire Wire Line
+	2300 7150 2300 7200
+Wire Wire Line
+	2850 7550 2300 7550
+Wire Wire Line
+	2300 7550 2300 7450
+Text GLabel 3750 7300 2    50   Input ~ 0
+EN_PACK_SENSE
+Wire Wire Line
+	3750 7300 3450 7300
+Connection ~ 3450 7300
+Text GLabel 1500 7200 0    50   Output ~ 0
+PACK_SENSE
+Wire Wire Line
+	2300 7200 1800 7200
+Connection ~ 2300 7200
+Wire Wire Line
+	2300 7200 2300 7250
+$Comp
+L Device:C_Small C309
+U 1 1 5F2113EB
+P 1800 7350
+F 0 "C309" H 1600 7400 50  0000 C CNN
+F 1 "100n" H 1600 7300 50  0000 C CNN
+F 2 "Capacitor_SMD:C_0603_1608Metric_Pad1.05x0.95mm_HandSolder" H 1800 7350 50  0001 C CNN
+F 3 "~" H 1800 7350 50  0001 C CNN
+	1    1800 7350
+	1    0    0    -1
+$EndComp
+Wire Wire Line
+	1800 7250 1800 7200
+Connection ~ 1800 7200
+Wire Wire Line
+	1800 7200 1500 7200
+Wire Wire Line
+	2300 7550 1800 7550
+Wire Wire Line
+	1800 7550 1800 7450
+Connection ~ 2300 7550
+$Comp
+L Device:Q_PMOS_GDS Q309
+U 1 1 5F227964
+P 7750 3550
+F 0 "Q309" H 7956 3504 50  0000 L CNN
+F 1 "FDD4685-F085" H 7956 3595 50  0000 L CNN
+F 2 "Package_TO_SOT_SMD:TO-252-2" H 7950 3650 50  0001 C CNN
+F 3 "~" H 7750 3550 50  0001 C CNN
+	1    7750 3550
+	1    0    0    1
+$EndComp
+Connection ~ 7850 3750
+Connection ~ 7850 3350
+Text Notes 600  7100 0    50   ~ 0
+1,64V bei 18V Eingangsspannung
 $EndSCHEMATC

Commit message: 3v3 regler ändern
Parts:
- F301: footprint Fuse:Fuseholder_Cylinder-5x20mm_Schurter_0031-8002_Horizontal_Open -> Fuse:Fuseholder_Cylinder-5x20mm_Schurter_0031_8201_Horizontal_Open
Changed lines of the file:
@@
 F 0 "F301" H 1850 6335 50  0000 C CNN
 F 1 "Fuse_Small" H 1850 6244 50  0000 C CNN
-F 2 "Fuse:Fuseholder_Cylinder-5x20mm_Schurter_0031-8002_Horizontal_Open" H 1850 6150 50  0001 C CNN
+F 2 "Fuse:Fuseholder_Cylinder-5x20mm_Schurter_0031_8201_Horizontal_Open" H 1850 6150 50  0001 C CNN
 F 3 "~" H 1850 6150 50  0001 C CNN
 	1    1850 6150

Commit message: TODO: power on detect einfügen
Parts:
- removed C304: 560u 50V, Capacitor_THT:CP_Radial_D12.5mm_P5.00mm, symbol Device:CP_Small
- added C304: 68u, Capacitor_THT:CP_Radial_D5.0mm_P2.50mm, symbol Device:CP1_Small
- added C?: 100n, Capacitor_SMD:C_0603_1608Metric_Pad1.05x0.95mm_HandSolder, symbol Device:C_Small
- R_CSB401: value 68m -> 200m
- renumbered Rcss401 to R_CSS401
Connections:
- net CHARGER_IOUT: now also C?.1
- net GND: now also C304.2, C?.2
- net POWER_SUPPLY: now also C304.1
Changed lines of the file:
@@
 $EndComp
 $Comp
-L Device:R_Small Rcss401
+L Device:R_Small R_CSS401
 U 1 1 5E73D449
 P 7850 3100
-F 0 "Rcss401" H 7909 3146 50  0000 L CNN
+F 0 "R_CSS401" H 7909 3146 50  0000 L CNN
 F 1 "33m" H 7909 3055 50  0000 L CNN
 F 2 "Resistor_SMD:R_1206_3216Metric_Pad1.42x1.75mm_HandSolder" H 7850 3100 50  0001 C CNN
@@
 P 8350 3950
 F 0 "R_CSB401" V 8450 3900 50  0000 C CNN
-F 1 "68m" V 8250 3950 50  0000 C CNN
+F 1 "200m" V 8250 3950 50  0000 C CNN
 F 2 "Resistor_SMD:R_1206_3216Metric_Pad1.42x1.75mm_HandSolder" H 8350 3950 50  0001 C CNN
 F 3 "~" H 8350 3950 50  0001 C CNN
@@
 Wire Wire Line
 	3800 3950 3600 3950
-$Comp
-L Device:CP_Small C?
-U 1 1 5ED2EE33
-P 4950 2450
-AR Path="/5E751A81/5ED2EE33" Ref="C?"  Part="1"
-AR Path="/5E73BAE8/5ED2EE33" Ref="C?"  Part="1"
-AR Path="/5E73BB4A/5ED2EE33" Ref="C304"  Part="1"
-F 0 "C304" H 5100 2550 50  0000 L CNN
-F 1 "560u 50V" H 5100 2400 50  0000 L CNN
-F 2 "Capacitor_THT:CP_Radial_D12.5mm_P5.00mm" H 4950 2450 50  0001 C CNN
-F 3 "https://www.mouser.de/datasheet/2/420/United-Chemi-Con-1109128.pdf" H 4950 2450 50  0001 C CNN
-	1    4950 2450
-	1    0    0    -1
-$EndComp
 Wire Wire Line
 	4950 2350 4950 2200
@@
 Text Notes 600  7100 0    50   ~ 0
 1,64V bei 18V Eingangsspannung
+$Comp
+L Device:CP1_Small C304
+U 1 1 5ED25F5D
+P 4950 2450
+F 0 "C304" H 5041 2496 50  0000 L CNN
+F 1 "68u" H 5041 2405 50  0000 L CNN
+F 2 "Capacitor_THT:CP_Radial_D5.0mm_P2.50mm" H 4950 2450 50  0001 C CNN
+F 3 "~" H 4950 2450 50  0001 C CNN
+	1    4950 2450
+	1    0    0    -1
+$EndComp
+$Comp
+L Device:C_Small C?
+U 1 1 5ED2EDE0
+P 2650 4300
+F 0 "C?" H 2800 4400 50  0000 C CNN
+F 1 "100n" H 2850 4300 50  0000 C CNN
+F 2 "Capacitor_SMD:C_0603_1608Metric_Pad1.05x0.95mm_HandSolder" H 2650 4300 50  0001 C CNN
+F 3 "~" H 2650 4300 50  0001 C CNN
+	1    2650 4300
+	1    0    0    -1
+$EndComp
+Wire Wire Line
+	2650 4200 2650 3950
+Wire Wire Line
+	2650 3950 2250 3950
+$Comp
+L power:GND #PWR?
+U 1 1 5ED36D0B
+P 2650 4600
+F 0 "#PWR?" H 2650 4350 50  0001 C CNN
+F 1 "GND" H 2655 4427 50  0000 C CNN
+F 2 "" H 2650 4600 50  0001 C CNN
+F 3 "" H 2650 4600 50  0001 C CNN
+	1    2650 4600
+	1    0    0    -1
+$EndComp
+Wire Wire Line
+	2650 4400 2650 4600
 $EndSCHEMATC

Commit message: 3v3 regler layout fertig
Parts:
- gave numbers to parts that had none: 1
Changed lines of the file:
@@
 $EndComp
 $Comp
-L Device:C_Small C?
+L Device:C_Small C301
 U 1 1 5ED2EDE0
 P 2650 4300
-F 0 "C?" H 2800 4400 50  0000 C CNN
+F 0 "C301" H 2800 4400 50  0000 C CNN
 F 1 "100n" H 2850 4300 50  0000 C CNN
 F 2 "Capacitor_SMD:C_0603_1608Metric_Pad1.05x0.95mm_HandSolder" H 2650 4300 50  0001 C CNN
@@
 	2650 3950 2250 3950
 $Comp
-L power:GND #PWR?
+L power:GND #PWR0307
 U 1 1 5ED36D0B
 P 2650 4600
-F 0 "#PWR?" H 2650 4350 50  0001 C CNN
+F 0 "#PWR0307" H 2650 4350 50  0001 C CNN
 F 1 "GND" H 2655 4427 50  0000 C CNN
 F 2 "" H 2650 4600 50  0001 C CNN
