File: 02_StepUp.sch (KiCad schematic (older format))
At the start: 29 parts, among them J301 Conn_02x04_Odd_Even, J302 Conn_02x04_Odd_Even, Q301 MMBT2222LT1G, Q302 TK7R7P10PL, U301 L7812, U302 UC3843_SOIC8

Commit message: Fertig zum letzten Check vor Bestellung
Parts:
- C304: footprint Capacitor_SMD:CP_Elec_5x5.4 -> Capacitor_THT:CP_Radial_D5.0mm_P2.50mm
Changed lines of the file:
@@
 F 0 "C304" H 4992 3046 50  0000 L CNN
 F 1 "25uF" H 4992 2955 50  0000 L CNN
-F 2 "Capacitor_SMD:CP_Elec_5x5.4" H 4900 3000 50  0001 C CNN
+F 2 "Capacitor_THT:CP_Radial_D5.0mm_P2.50mm" H 4900 3000 50  0001 C CNN
 F 3 "~" H 4900 3000 50  0001 C CNN
 	1    4900 3000

Commit message: Board abgeschickt
Parts:
- added C309: 100nF, Capacitor_SMD:C_0603_1608Metric_Pad1.05x0.95mm_HandSolder, symbol Device:C_Small
- C302: value 1n2 -> 1.2nF
- C303: value 100n -> 100nF
- C306: value C_Small -> 100nF
- L301: value 10uH PQ2617BHA-100K -> 10uH PQ2617BLA-100K
Connections:
- wire segments 102 -> 104
Changed lines of the file:
@@
 P 5250 3600
 F 0 "U302" H 5350 4150 50  0000 C CNN
-F 1 "UC3843_SOIC8" H 5600 4000 50  0000 C CNN
+F 1 "UC3843_SOIC8" H 5350 3650 50  0000 C CNN
 F 2 "Package_SO:SOIC-8_3.9x4.9mm_P1.27mm" H 5250 3150 50  0001 C CNN
 F 3 "http://www.ti.com/lit/ds/symlink/uc3842.pdf" H 5250 3600 50  0001 C CNN
@@
 P 6550 2900
 F 0 "L301" H 6598 2946 50  0000 L CNN
-F 1 "10uH PQ2617BHA-100K " H 6598 2855 50  0000 L CNN
+F 1 "10uH PQ2617BLA-100K " H 6598 2855 50  0000 L CNN
 F 2 "Inductor_SMD:PQ2617BHA-330K" H 6550 2900 50  0001 C CNN
 F 3 "https://www.mouser.de/datasheet/2/54/bourns_PQ2617BHA_datasheet-1159314.pdf" H 6550 2900 50  0001 C CNN
@@
 P 4600 3850
 F 0 "C303" H 4400 3950 50  0000 L CNN
-F 1 "100n" H 4400 3750 50  0000 L CNN
+F 1 "100nF" H 4400 3750 50  0000 L CNN
 F 2 "Capacitor_SMD:C_0603_1608Metric_Pad1.05x0.95mm_HandSolder" H 4600 3850 50  0001 C CNN
 F 3 "~" H 4600 3850 50  0001 C CNN
@@
 P 4000 3850
 F 0 "C302" H 4092 3896 50  0000 L CNN
-F 1 "1n2" H 4092 3805 50  0000 L CNN
+F 1 "1.2nF" H 4092 3805 50  0000 L CNN
 F 2 "Capacitor_SMD:C_0603_1608Metric_Pad1.05x0.95mm_HandSolder" H 4000 3850 50  0001 C CNN
 F 3 "~" H 4000 3850 50  0001 C CNN
@@
 P 2800 3850
 F 0 "C306" H 2892 3896 50  0000 L CNN
-F 1 "C_Small" H 2892 3805 50  0000 L CNN
+F 1 "100nF" H 2892 3805 50  0000 L CNN
 F 2 "Capacitor_SMD:C_0603_1608Metric_Pad1.05x0.95mm_HandSolder" H 2800 3850 50  0001 C CNN
 F 3 "~" H 2800 3850 50  0001 C CNN
@@
 Wire Wire Line
 	5450 2600 6050 2600
+$Comp
+L Device:C_Small C309
+U 1 1 5EB3CDC2
+P 5550 3000
+F 0 "C309" H 5642 3046 50  0000 L CNN
+F 1 "100nF" H 5642 2955 50  0000 L CNN
+F 2 "Capacitor_SMD:C_0603_1608Metric_Pad1.05x0.95mm_HandSolder" H 5550 3000 50  0001 C CNN
+F 3 "~" H 5550 3000 50  0001 C CNN
+	1    5550 3000
+	1    0    0    -1
+$EndComp
+Wire Wire Line
+	5550 2900 5550 2800
+Wire Wire Line
+	5550 2800 5250 2800
+Connection ~ 5250 2800
+$Comp
+L power:GNDPWR #PWR0301
+U 1 1 5EB40078
+P 5550 3100
+F 0 "#PWR0301" H 5550 2900 50  0001 C CNN
+F 1 "GNDPWR" H 5554 2946 50  0000 C CNN
+F 2 "" H 5550 3050 50  0001 C CNN
+F 3 "" H 5550 3050 50  0001 C CNN
+	1    5550 3100
+	1    0    0    -1
+$EndComp
 $EndSCHEMATC

Commit message: mute and stdby tda7498 geändert, tda7418 durch tda7719 ersetzt, xs3868 durch bk8000l ersetzt, 3v3 stepdown statt LDO. BMS gelöscht.  TODO: Möglichkeit stepup und stepdown als modul aufzusetzen
Parts:
- removed C304: 25uF, Capacitor_THT:CP_Radial_D5.0mm_P2.50mm, symbol Device:C_Small
- removed C309: 100nF, Capacitor_SMD:C_0603_1608Metric_Pad1.05x0.95mm_HandSolder, symbol Device:C_Small
- removed D301: STPS2045C, Package_TO_SOT_SMD:TO-263-2, symbol Device:D_Schottky_x2_KCom_AKA
- removed HS303, HS304: 573300D00000G, Heatsink:Heatsink_AAVID_573300D00010G_TO-263, symbol Mechanical:Heatsink_Pad
- removed U301: L7812, Package_TO_SOT_SMD:TO-263-2, symbol Regulator_Linear:L7812
- added C201, C203: 68u, Capacitor_THT:CP_Radial_D6.3mm_P2.50mm, symbol Device:CP1_Small
- added C202: 100n, Capacitor_SMD:C_0603_1608Metric_Pad1.05x0.95mm_HandSolder, symbol Device:C_Small
- added D201: STPS1045B-TR, Package_TO_SOT_SMD:TO-252-2, symbol Device:D_Schottky_x2_KCom_AKA
- added J201: Conn_02x01, Connector_PinHeader_2.54mm:PinHeader_1x02_P2.54mm_Vertical, symbol Connector_Generic:Conn_02x01
- added R201, R203, R204, R205: 10K, Resistor_SMD:R_0603_1608Metric_Pad1.05x0.95mm_HandSolder, symbol Device:R_Small
- added R202: 47K, Resistor_SMD:R_0603_1608Metric_Pad1.05x0.95mm_HandSolder, symbol Device:R_Small
- added R206: 0R, Resistor_SMD:R_0603_1608Metric_Pad1.05x0.95mm_HandSolder, symbol Device:R_Small
- added U201: XC6216C, Package_TO_SOT_SMD:SOT-23-5_HandSoldering, symbol Regulator_Linear:XC6216C
- C306: value 100nF -> 220nF
- L301: value 10uH PQ2617BLA-100K -> 33uH PQ2617BLA-330K
- Q302: footprint Package_TO_SOT_SMD:TO-263-2 -> Package_TO_SOT_SMD:TO-252-2
- R303: value 30K -> 10K
Connections:
- net labels added: 12V, ENABLE_12V, GND, IN_STEPUP, STEPUP_CS, STEPUP_GND, STPUP_GND
- wire segments 104 -> 116
Other:
- note added: "Timing Cap so nah wie möglich am IC (Single Ground Point)!"
- moved on the sheet: C301, C302, C303, C305, C306, C307, C308, HS301, HS302, J301, J302, L301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

Commit message: neue schematic fertig zum rewiew. DRC clean
Connections:
- wire segments 116 -> 121
Other:
- moved on the sheet: R308, R309, RV301
Changed lines of the file:
@@
 L Device:R_Small R308
 U 1 1 5E7975A3
-P 8700 5450
-F 0 "R308" H 8641 5404 50  0000 R CNN
-F 1 "2K94" H 8641 5495 50  0000 R CNN
-F 2 "Resistor_SMD:R_0603_1608Metric_Pad1.05x0.95mm_HandSolder" H 8700 5450 50  0001 C CNN
-F 3 "~" H 8700 5450 50  0001 C CNN
-	1    8700 5450
+P 9100 5450
+F 0 "R308" H 9041 5404 50  0000 R CNN
+F 1 "2K94" H 9041 5495 50  0000 R CNN
+F 2 "Resistor_SMD:R_0603_1608Metric_Pad1.05x0.95mm_HandSolder" H 9100 5450 50  0001 C CNN
+F 3 "~" H 9100 5450 50  0001 C CNN
+	1    9100 5450
 	-1   0    0    1
 $EndComp
@@
 L Device:R_Small R309
 U 1 1 5E79763C
-P 8700 5750
-F 0 "R309" H 8641 5704 50  0000 R CNN
-F 1 "1K" H 8641 5795 50  0000 R CNN
-F 2 "Resistor_SMD:R_0603_1608Metric_Pad1.05x0.95mm_HandSolder" H 8700 5750 50  0001 C CNN
-F 3 "~" H 8700 5750 50  0001 C CNN
-	1    8700 5750
+P 9100 5750
+F 0 "R309" H 9041 5704 50  0000 R CNN
+F 1 "1K" H 9041 5795 50  0000 R CNN
+F 2 "Resistor_SMD:R_0603_1608Metric_Pad1.05x0.95mm_HandSolder" H 9100 5750 50  0001 C CNN
+F 3 "~" H 9100 5750 50  0001 C CNN
+	1    9100 5750
 	-1   0    0    1
 $EndComp
 Wire Wire Line
-	8700 5650 8700 5600
-Wire Wire Line
-	8700 5350 8700 5300
-Wire Wire Line
-	8700 5900 8700 5850
-Wire Wire Line
-	8700 4950 8700 4850
+	9100 5350 9100 5300
+Wire Wire Line
+	9100 5900 9100 5850
+Wire Wire Line
+	9100 4950 9100 4850
 Wire Wire Line
 	8700 4850 8400 4850
@@
 Wire Wire Line
 	4700 5350 4550 5350
-Connection ~ 8700 5600
-Wire Wire Line
-	8700 5600 8700 5550
 Text Label 4700 5800 0    50   ~ 0
 FB_BOOST
@@
 Wire Wire Line
 	3500 1750 3500 1650
-$Comp
-L power:GNDPWR #PWR0126
-U 1 1 5E7ACC52
-P 3500 1950
-F 0 "#PWR0126" H 3500 1750 50  0001 C CNN
-F 1 "GNDPWR" H 3504 1796 50  0000 C CNN
-F 2 "" H 3500 1900 50  0001 C CNN
-F 3 "" H 3500 1900 50  0001 C CNN
-	1    3500 1950
-	1    0    0    -1
-$EndComp
 $Comp
 L power:GNDPWR #PWR0128
@@
 L Device:R_POT RV301
 U 1 1 5EEEB2DA
-P 8700 5100
-F 0 "RV301" H 8630 5146 50  0000 R CNN
-F 1 "10K" H 8630 5055 50  0000 R CNN
-F 2 "Potentiometer_SMD:Potentiometer_Bourns_3314J_Vertical" H 8700 5100 50  0001 C CNN
-F 3 "https://www.mouser.de/datasheet/2/54/tc33-778219.pdf" H 8700 5100 50  0001 C CNN
-	1    8700 5100
-	1    0    0    -1
-$EndComp
-Wire Wire Line
-	8850 5100 8900 5100
-Wire Wire Line
-	8900 5100 8900 5300
-Wire Wire Line
-	8900 5300 8700 5300
-Connection ~ 8700 5300
-Wire Wire Line
-	8700 5300 8700 5250
+P 9100 5100
+F 0 "RV301" H 9030 5146 50  0000 R CNN
+F 1 "10K" H 9030 5055 50  0000 R CNN
+F 2 "Potentiometer_SMD:Potentiometer_Bourns_3314J_Vertical" H 9100 5100 50  0001 C CNN
+F 3 "https://www.mouser.de/datasheet/2/54/tc33-778219.pdf" H 9100 5100 50  0001 C CNN
+	1    9100 5100
+	1    0    0    -1
+$EndComp
+Wire Wire Line
+	9250 5100 9300 5100
+Wire Wire Line
+	9300 5100 9300 5300
+Wire Wire Line
+	9300 5300 9100 5300
+Connection ~ 9100 5300
+Wire Wire Line
+	9100 5300 9100 5250
 $Comp
 L Device:CP_Small C?
@@
 	2150 1650 1550 1650
 Wire Wire Line
-	8700 4850 9250 4850
+	8700 4850 9100 4850
 Wire Wire Line
 	9950 4850 9750 4850
@@
 Wire Wire Line
 	5200 5900 3950 5900
-Connection ~ 3500 1950
 Wire Wire Line
 	4650 4950 4700 4950
@@
 Text Label 5700 1650 0    50   ~ 0
 IN_STEPUP
-Text Label 9200 5600 0    50   ~ 0
+Text Label 8950 5600 2    50   ~ 0
 FB_BOOST
 Wire Wire Line
-	9200 5600 8700 5600
-Wire Wire Line
 	6850 4850 7350 4850
 Wire Wire Line
 	7900 4850 8200 4850
-Text Label 5750 5500 0    50   ~ 0
+Text Label 6100 5650 2    50   ~ 0
 STEPUP_CS
-Text Label 2900 6000 0    50   ~ 0
+Text Label 3750 6000 0    50   ~ 0
 STEPUP_CS
 Wire Wire Line
@@
 	2750 6000 3550 6000
 Wire Wire Line
-	5700 5500 6300 5500
+	5700 5500 6200 5500
 Text Label 2950 4950 0    50   ~ 0
 IN_STEPUP
@@
 Text Label 5650 5900 0    50   ~ 0
 STEPUP_GND
-Wire Wire Line
-	5650 5900 5500 5900
 Connection ~ 5200 5900
 $Comp
 L power:GND #PWR0209
 U 1 1 5EEA9D8A
-P 8700 5900
-F 0 "#PWR0209" H 8700 5650 50  0001 C CNN
-F 1 "GND" H 8705 5727 50  0000 C CNN
-F 2 "" H 8700 5900 50  0001 C CNN
-F 3 "" H 8700 5900 50  0001 C CNN
-	1    8700 5900
+P 9100 5900
+F 0 "#PWR0209" H 9100 5650 50  0001 C CNN
+F 1 "GND" H 9105 5727 50  0000 C CNN
+F 2 "" H 9100 5900 50  0001 C CNN
+F 3 "" H 9100 5900 50  0001 C CNN
+	1    9100 5900
 	1    0    0    -1
 $EndComp
@@
 F 3 "" H 8200 5900 50  0001 C CNN
 	1    8200 5900
-	1    0    0    -1
-$EndComp
-$Comp
-L power:GND #PWR0207
-U 1 1 5EEA9E33
-P 6850 5900
-F 0 "#PWR0207" H 6850 5650 50  0001 C CNN
-F 1 "GND" H 6855 5727 50  0000 C CNN
-F 2 "" H 6850 5900 50  0001 C CNN
-F 3 "" H 6850 5900 50  0001 C CNN
-	1    6850 5900
 	1    0    0    -1
 $EndComp
@@
 	0    -1   -1   0
 $EndComp
+$Comp
+L power:GND #PWR?
+U 1 1 5F07DA47
+P 3500 1950
+AR Path="/5EA6895E/5F07DA47" Ref="#PWR?"  Part="1"
+AR Path="/5E73BAE8/5F07DA47" Ref="#PWR0207"  Part="1"
+F 0 "#PWR0207" H 3500 1700 50  0001 C CNN
+F 1 "GND" H 3505 1777 50  0000 C CNN
+F 2 "" H 3500 1950 50  0001 C CNN
+F 3 "" H 3500 1950 50  0001 C CNN
+	1    3500 1950
+	1    0    0    -1
+$EndComp
+Connection ~ 3500 1950
+Wire Wire Line
+	3750 6000 3550 6000
+Connection ~ 3550 6000
+Wire Wire Line
+	6200 5500 6200 5650
+Wire Wire Line
+	6200 5650 6100 5650
+Connection ~ 6200 5500
+Wire Wire Line
+	6200 5500 6300 5500
+Connection ~ 9100 4850
+Wire Wire Line
+	9100 4850 9250 4850
+Wire Wire Line
+	9100 5550 9100 5600
+Wire Wire Line
+	8950 5600 9100 5600
+Connection ~ 9100 5600
+Wire Wire Line
+	9100 5600 9100 5650
+Wire Wire Line
+	5500 5900 6850 5900
 $EndSCHEMATC

Commit message: module, falls schaltung nicht funktioniert hinzugefügt
Parts:
- added U202: StepUp, Module:StepUpModul, symbol MySymbols:StepUp
- renumbered C203 to C_1, C303 to C_2, C306 to C_3, C302 to C_4, C307 to C_5_1, C301 to C_5_2, C201 to C_5_3, C308 to C_6_1, C305 to C_6_2, D201 to D_1, RV301 to RV_1, R201 to R_10, R202 to R_11, R203 to R_12, R308 to R_2, R309 to R_3, R303 to R_4_1, R205 to R_4_2, R204 to R_4_3, R305 to R_5, R302 to R_6, R301 to R_7, R306 to R_8, R304 to R_9, Q301 to S_1, Q302 to S_2, U302 to U_2
Other:
- note added: "Möglichkeit fertigen StepUp aufzusetzen"

Commit message: 3v3 regler layout fertig
Parts:
- removed C_5_3: 68u, Capacitor_THT:CP_Radial_D6.3mm_P2.50mm, symbol Device:CP1_Small
- added C201: 100n, Capacitor_SMD:C_0603_1608Metric_Pad1.05x0.95mm_HandSolder, symbol Device:C_Small
Changed lines of the file:
@@
-$EndComp
-$Comp
-L Device:CP1_Small C?
-U 1 1 5EE9A404
-P 2600 3350
-AR Path="/5E73BB4A/5EE9A404" Ref="C?"  Part="1"
-AR Path="/5ED2496F/5EE9A404" Ref="C?"  Part="1"
-AR Path="/5E73BAE8/5EE9A404" Ref="C_5_3"  Part="1"
-F 0 "C_5_3" H 2691 3396 50  0000 L CNN
-F 1 "68u" H 2691 3305 50  0000 L CNN
-F 2 "Capacitor_THT:CP_Radial_D6.3mm_P2.50mm" H 2600 3350 50  0001 C CNN
-F 3 "~" H 2600 3350 50  0001 C CNN
-	1    2600 3350
-	1    0    0    -1
 $EndComp
 $Comp
@@
 Text Notes 8350 1950 0    50   ~ 0
 Möglichkeit fertigen StepUp aufzusetzen
+$Comp
+L Device:C_Small C201
+U 1 1 5ED41E8D
+P 2600 3350
+F 0 "C201" H 2300 3400 50  0000 L CNN
+F 1 "100n" H 2250 3300 50  0000 L CNN
+F 2 "Capacitor_SMD:C_0603_1608Metric_Pad1.05x0.95mm_HandSolder" H 2600 3350 50  0001 C CNN
+F 3 "~" H 2600 3350 50  0001 C CNN
+	1    2600 3350
+	1    0    0    -1
+$EndComp
 $EndSCHEMATC

Commit message: vor änderungen von der Arbeit
Parts:
- R206: footprint Resistor_SMD:R_0603_1608Metric_Pad1.05x0.95mm_HandSolder -> Resistor_SMD:R_1206_3216Metric_Pad1.42x1.75mm_HandSolder
- U201: symbol Regulator_Linear:XC6216C -> MukkeBox-rescue:XC6216C-Regulator_Linear
- U202: symbol MySymbols:StepUp -> MukkeBox-rescue:StepUp-MySymbols
- U_2: symbol Regulator_Controller:UC3843_SOIC8 -> MukkeBox-rescue:UC3843_SOIC8-Regulator_Controller
Connections:
- net labels removed: GNDPWR, STPUP_GND
Changed lines of the file:
@@
 UC1842 Step Up von aliexpress yo\nhttps://www.360customs.de/2014/05/103050100w-led-applikation-treiber/?cookie-state-change=1586628857397\n
 $Comp
-L Regulator_Controller:UC3843_SOIC8 U_2
+L MukkeBox-rescue:UC3843_SOIC8-Regulator_Controller U_2
 U 1 1 5E7948D1
 P 5200 5300
@@
 Wire Wire Line
 	3500 1750 3500 1650
-$Comp
-L power:GNDPWR #PWR0128
-U 1 1 5E7AEF97
-P 6050 4700
-F 0 "#PWR0128" H 6050 4500 50  0001 C CNN
-F 1 "GNDPWR" V 6150 4650 50  0000 C CNN
-F 2 "" H 6050 4650 50  0001 C CNN
-F 3 "" H 6050 4650 50  0001 C CNN
-	1    6050 4700
-	0    -1   -1   0
-$EndComp
 Text GLabel 9950 4850 2    50   Output ~ 0
 POWER_AMP
@@
 Connection ~ 4550 5600
 $Comp
-L Regulator_Linear:XC6216C U?
+L MukkeBox-rescue:XC6216C-Regulator_Linear U?
 U 1 1 5ECF85A5
 P 4250 3200
@@
 Wire Wire Line
 	5200 4600 5200 4550
-Text Label 4750 4600 2    50   ~ 0
-STPUP_GND
 Wire Wire Line
 	4900 4600 4750 4600
-Text Label 4450 4950 2    50   ~ 0
-STPUP_GND
 Text Label 5650 5900 0    50   ~ 0
 STEPUP_GND
 Connection ~ 5200 5900
-$Comp
-L power:GND #PWR0209
-U 1 1 5EEA9D8A
-P 9100 5900
-F 0 "#PWR0209" H 9100 5650 50  0001 C CNN
-F 1 "GND" H 9105 5727 50  0000 C CNN
-F 2 "" H 9100 5900 50  0001 C CNN
-F 3 "" H 9100 5900 50  0001 C CNN
-	1    9100 5900
-	1    0    0    -1
-$EndComp
 $Comp
 L power:GND #PWR0208
@@
 F 0 "R206" H 5559 6096 50  0000 L CNN
 F 1 "0R" H 5559 6005 50  0000 L CNN
-F 2 "Resistor_SMD:R_0603_1608Metric_Pad1.05x0.95mm_HandSolder" H 5500 6050 50  0001 C CNN
+F 2 "Resistor_SMD:R_1206_3216Metric_Pad1.42x1.75mm_HandSolder" H 5500 6050 50  0001 C CNN
 F 3 "~" H 5500 6050 50  0001 C CNN
 	1    5500 6050
@@
 	5500 5900 6850 5900
 $Comp
-L MySymbols:StepUp U202
+L MukkeBox-rescue:StepUp-MySymbols U202
 U 1 1 5FE6AEE3
 P 8900 2400
@@
 	1    0    0    -1
 $EndComp
+Text Label 4750 4600 2    50   ~ 0
+STEPUP_GND
+Text Label 4450 4950 2    50   ~ 0
+STEPUP_GND
+Text Label 6050 4700 0    50   ~ 0
+STEPUP_GND
+Text Label 9100 5900 0    50   ~ 0
+STEPUP_GND
 $EndSCHEMATC
