File: 02_StepUp.sch (KiCad schematic (older format))
At the start: 30 parts, among them J301 Conn_02x04_Odd_Even, J302 Conn_02x04_Odd_Even, Q201 CSD18504Q5A, U201 STPS30M60DJF, U202 StepUp, U203 TPS40210

Commit message: Charger ausgetauscht, Mosfet und Dioden durch billigere ersetzt
Parts:
- removed U201: STPS30M60DJF, Package_TO_SOT_SMD:TDSON-8-1_HandSoldering, symbol MukkeBox-rescue:Diode-TDSON-8-MySymbols
- added D201: PS1060L, Package_TO_SOT_SMD:TO-277B, symbol Device:PS1060L
- added Q202: VS6412AE, Package_SON:Diodes_PowerDI3333-8, symbol Transistor_FET:CSD18504Q5A
- Q201: value CSD18504Q5A -> VS6412AE; footprint Package_TO_SOT_SMD:TDSON-8-1_HandSoldering -> Package_SON:Diodes_PowerDI3333-8
Connections:
- wire segments 106 -> 108
Other:
- note added: "CSD18504Q5A\nIPC50N04S5L5R5ATMA1\nBSC067N06LS3 G"
- note removed: "IPC50N04S5L5R5ATMA1\nBSC067N06LS3 G"
- moved on the sheet: R203, R_8
Changed lines of the file:
@@
 EESchema Schematic File Version 4
-EELAYER 30 0
+LIBS:MukkeBox-cache
+EELAYER 26 0
 EELAYER END
 $Descr A4 11693 8268
@@
 L Device:R_Small R_8
 U 1 1 5E7965D6
-P 6700 4500
-F 0 "R_8" H 6641 4454 50  0000 R CNN
-F 1 "R007" H 6641 4545 50  0000 R CNN
-F 2 "Resistor_SMD:R_2010_5025Metric_Pad1.52x2.65mm_HandSolder" H 6700 4500 50  0001 C CNN
-F 3 "~" H 6700 4500 50  0001 C CNN
-	1    6700 4500
+P 6950 4550
+F 0 "R_8" H 6891 4504 50  0000 R CNN
+F 1 "R007" H 6891 4595 50  0000 R CNN
+F 2 "Resistor_SMD:R_2010_5025Metric_Pad1.52x2.65mm_HandSolder" H 6950 4550 50  0001 C CNN
+F 3 "~" H 6950 4550 50  0001 C CNN
+	1    6950 4550
 	-1   0    0    1
 $EndComp
@@
 	6700 3550 7200 3550
 Wire Wire Line
-	7900 3550 8050 3550
-Wire Wire Line
 	6700 3600 6700 3550
 Connection ~ 6700 3550
@@
 U 1 1 5EEA1196
 P 6150 3800
-F 0 "R204" V 6250 3800 50  0000 C CNN
-F 1 "22R" V 6350 3800 50  0000 C CNN
+F 0 "R204" V 5950 3800 50  0000 C CNN
+F 1 "22R" V 6050 3800 50  0000 C CNN
 F 2 "Resistor_SMD:R_0603_1608Metric_Pad1.05x0.95mm_HandSolder" H 6150 3800 50  0001 C CNN
 F 3 "~" H 6150 3800 50  0001 C CNN
@@
 	0    1    1    0
 $EndComp
-Wire Wire Line
-	6400 3800 6350 3800
 $Comp
 L Device:C_Small C208
@@
 	0    1    1    0
 $EndComp
-Wire Wire Line
-	6050 3800 5950 3800
 $Comp
 L power:GND #PWR0214
 U 1 1 5EEC344A
-P 6700 4600
-F 0 "#PWR0214" H 6700 4350 50  0001 C CNN
-F 1 "GND" H 6705 4427 50  0000 C CNN
-F 2 "" H 6700 4600 50  0001 C CNN
-F 3 "" H 6700 4600 50  0001 C CNN
-	1    6700 4600
+P 6950 4650
+F 0 "#PWR0214" H 6950 4400 50  0001 C CNN
+F 1 "GND" H 6955 4477 50  0000 C CNN
+F 2 "" H 6950 4650 50  0001 C CNN
+F 3 "" H 6950 4650 50  0001 C CNN
+	1    6950 4650
 	1    0    0    -1
 $EndComp
@@
 	6700 4200 6250 4200
 Connection ~ 6700 4200
-Wire Wire Line
-	6700 4200 6700 4400
 Wire Wire Line
 	6050 4200 5700 4200
@@
 L Device:R_Small R203
 U 1 1 5EFF1EE0
-P 6150 3700
-F 0 "R203" V 6250 3700 50  0000 C CNN
-F 1 "22R" V 6350 3700 50  0000 C CNN
-F 2 "Resistor_SMD:R_0603_1608Metric_Pad1.05x0.95mm_HandSolder" H 6150 3700 50  0001 C CNN
-F 3 "~" H 6150 3700 50  0001 C CNN
-	1    6150 3700
+P 6400 4100
+F 0 "R203" V 6500 4100 50  0000 C CNN
+F 1 "22R" V 6600 4100 50  0000 C CNN
+F 2 "Resistor_SMD:R_0603_1608Metric_Pad1.05x0.95mm_HandSolder" H 6400 4100 50  0001 C CNN
+F 3 "~" H 6400 4100 50  0001 C CNN
+	1    6400 4100
 	0    -1   -1   0
 $EndComp
-Wire Wire Line
-	6250 3700 6350 3700
-Wire Wire Line
-	6350 3700 6350 3800
-Connection ~ 6350 3800
-Wire Wire Line
-	6350 3800 6250 3800
-Wire Wire Line
-	6050 3700 5950 3700
-Wire Wire Line
-	5950 3700 5950 3800
-Connection ~ 5950 3800
-Wire Wire Line
-	5950 3800 4750 3800
 Text Notes 5800 4600 0    50   ~ 0
 180p
 Text Notes 6950 3450 1    50   ~ 0
 13-39uH
-Text Notes 6800 4150 0    50   ~ 0
+Text Notes 7950 5550 0    50   ~ 0
 50A
 Text Notes 7600 3200 0    50   ~ 0
@@
 Wire Wire Line
 	4850 4350 4850 4100
-$Comp
-L Transistor_FET:CSD18504Q5A Q201
-U 1 1 5ED2E926
-P 6600 3800
-F 0 "Q201" H 6806 3846 50  0000 L CNN
-F 1 "CSD18504Q5A" H 6806 3755 50  0000 L CNN
-F 2 "Package_TO_SOT_SMD:TDSON-8-1_HandSoldering" H 6800 3725 50  0001 L CIN
-F 3 "http://www.ti.com/lit/gpn/csd18504q5a" V 6600 3800 50  0001 L CNN
-	1    6600 3800
-	1    0    0    -1
-$EndComp
-Text Notes 6800 4050 0    50   ~ 0
-IPC50N04S5L5R5ATMA1\nBSC067N06LS3 G
+Text Notes 7950 5400 0    50   ~ 0
+CSD18504Q5A\nIPC50N04S5L5R5ATMA1\nBSC067N06LS3 G
 Text Notes 7450 2950 0    50   ~ 0
 STPS30M60DJF
-$Comp
-L MukkeBox-rescue:Diode-TDSON-8-MySymbols U201
-U 1 1 5ED46133
-P 7850 3550
-AR Path="/5ED46133" Ref="U201"  Part="1"
-AR Path="/5E73BAE8/5ED46133" Ref="U201"  Part="1"
-F 0 "U201" H 7650 3815 50  0000 C CNN
-F 1 "STPS30M60DJF" H 7650 3724 50  0000 C CNN
-F 2 "Package_TO_SOT_SMD:TDSON-8-1_HandSoldering" H 7850 3550 50  0001 C CNN
-F 3 "" H 7850 3550 50  0001 C CNN
-	1    7850 3550
-	1    0    0    -1
-$EndComp
-Wire Wire Line
-	7200 3550 7400 3550
 Wire Wire Line
 	8050 3550 8550 3550
+$Comp
+L Device:PS1060L D201
+U 1 1 5F75672E
+P 7650 3550
+F 0 "D201" H 7650 3325 50  0000 C CNN
+F 1 "PS1060L" H 7650 3416 50  0000 C CNN
+F 2 "Package_TO_SOT_SMD:TO-277B" H 7650 3550 50  0001 C CNN
+F 3 "https://datasheet.lcsc.com/szlcsc/1911251432_Chongqing-Pingwei-Tech-PS1060L_C432724.pdf" H 7650 3550 50  0001 C CNN
+	1    7650 3550
+	-1   0    0    1
+$EndComp
+Wire Wire Line
+	7800 3550 8050 3550
+Wire Wire Line
+	7200 3550 7500 3550
+$Comp
+L Transistor_FET:CSD18504Q5A Q201
+U 1 1 5F75D83F
+P 6600 3800
+AR Path="/5E73BAE8/5F75D83F" Ref="Q201"  Part="1"
+AR Path="/5E73BB4A/5F75D83F" Ref="Q?"  Part="1"
+F 0 "Q201" H 6806 3846 50  0000 L CNN
+F 1 "VS6412AE" H 6806 3755 50  0000 L CNN
+F 2 "Package_SON:Diodes_PowerDI3333-8" H 6800 3725 50  0001 L CIN
+F 3 "https://datasheet.lcsc.com/szlcsc/1909091006_Vanguard-VS6412AE_C427044.pdf" V 6600 3800 50  0001 L CNN
+	1    6600 3800
+	1    0    0    -1
+$EndComp
+$Comp
+L Transistor_FET:CSD18504Q5A Q202
+U 1 1 5F760DD5
+P 7100 4100
+AR Path="/5E73BAE8/5F760DD5" Ref="Q202"  Part="1"
+AR Path="/5E73BB4A/5F760DD5" Ref="Q?"  Part="1"
+F 0 "Q202" H 7306 4146 50  0000 L CNN
+F 1 "VS6412AE" H 7306 4055 50  0000 L CNN
+F 2 "Package_SON:Diodes_PowerDI3333-8" H 7300 4025 50  0001 L CIN
+F 3 "https://datasheet.lcsc.com/szlcsc/1909091006_Vanguard-VS6412AE_C427044.pdf" V 7100 4100 50  0001 L CNN
+	1    7100 4100
+	1    0    0    -1
+$EndComp
+Wire Wire Line
+	7200 3900 7200 3550
+Wire Wire Line
+	6250 3800 6400 3800
+Wire Wire Line
+	4750 3800 6000 3800
+Wire Wire Line
+	6900 4100 6500 4100
+Wire Wire Line
+	6300 4100 6000 4100
+Wire Wire Line
+	6000 4100 6000 3800
+Connection ~ 6000 3800
+Wire Wire Line
+	6000 3800 6050 3800
+Wire Wire Line
+	7200 4300 7200 4450
+Wire Wire Line
+	7200 4450 6950 4450
+Wire Wire Line
+	6700 4450 6950 4450
+Wire Wire Line
+	6700 4200 6700 4450
+Connection ~ 6950 4450
 $EndSCHEMATC

Commit message: Änderungen Arbeit hinzugefügt: Layout neuer Charger
Parts:
- removed Q202: VS6412AE, Package_SON:Diodes_PowerDI3333-8, symbol Transistor_FET:CSD18504Q5A
- D201: symbol Device:PS1060L -> MukkeBox-rescue:PS1060L-Device
Connections:
- wire segments 108 -> 106
Other:
- moved on the sheet: R203, R_8
Changed lines of the file:
@@
 EESchema Schematic File Version 4
-LIBS:MukkeBox-cache
-EELAYER 26 0
+EELAYER 30 0
 EELAYER END
 $Descr A4 11693 8268
@@
 L Device:R_Small R_8
 U 1 1 5E7965D6
-P 6950 4550
-F 0 "R_8" H 6891 4504 50  0000 R CNN
-F 1 "R007" H 6891 4595 50  0000 R CNN
-F 2 "Resistor_SMD:R_2010_5025Metric_Pad1.52x2.65mm_HandSolder" H 6950 4550 50  0001 C CNN
-F 3 "~" H 6950 4550 50  0001 C CNN
-	1    6950 4550
+P 6700 4550
+F 0 "R_8" H 6641 4504 50  0000 R CNN
+F 1 "R007" H 6641 4595 50  0000 R CNN
+F 2 "Resistor_SMD:R_2010_5025Metric_Pad1.52x2.65mm_HandSolder" H 6700 4550 50  0001 C CNN
+F 3 "~" H 6700 4550 50  0001 C CNN
+	1    6700 4550
 	-1   0    0    1
 $EndComp
@@
 P 6150 3800
 F 0 "R204" V 5950 3800 50  0000 C CNN
-F 1 "22R" V 6050 3800 50  0000 C CNN
+F 1 "22R" V 6400 3800 50  0000 C CNN
 F 2 "Resistor_SMD:R_0603_1608Metric_Pad1.05x0.95mm_HandSolder" H 6150 3800 50  0001 C CNN
 F 3 "~" H 6150 3800 50  0001 C CNN
@@
 L power:GND #PWR0214
 U 1 1 5EEC344A
-P 6950 4650
-F 0 "#PWR0214" H 6950 4400 50  0001 C CNN
-F 1 "GND" H 6955 4477 50  0000 C CNN
-F 2 "" H 6950 4650 50  0001 C CNN
-F 3 "" H 6950 4650 50  0001 C CNN
-	1    6950 4650
+P 6700 4650
+F 0 "#PWR0214" H 6700 4400 50  0001 C CNN
+F 1 "GND" H 6705 4477 50  0000 C CNN
+F 2 "" H 6700 4650 50  0001 C CNN
+F 3 "" H 6700 4650 50  0001 C CNN
+	1    6700 4650
 	1    0    0    -1
 $EndComp
@@
 L Device:R_Small R203
 U 1 1 5EFF1EE0
-P 6400 4100
-F 0 "R203" V 6500 4100 50  0000 C CNN
-F 1 "22R" V 6600 4100 50  0000 C CNN
-F 2 "Resistor_SMD:R_0603_1608Metric_Pad1.05x0.95mm_HandSolder" H 6400 4100 50  0001 C CNN
-F 3 "~" H 6400 4100 50  0001 C CNN
-	1    6400 4100
+P 6150 3900
+F 0 "R203" V 6050 3900 50  0000 C CNN
+F 1 "22R" V 6350 3900 50  0000 C CNN
+F 2 "Resistor_SMD:R_0603_1608Metric_Pad1.05x0.95mm_HandSolder" H 6150 3900 50  0001 C CNN
+F 3 "~" H 6150 3900 50  0001 C CNN
+	1    6150 3900
 	0    -1   -1   0
 $EndComp
@@
 	8050 3550 8550 3550
 $Comp
-L Device:PS1060L D201
+L MukkeBox-rescue:PS1060L-Device D201
 U 1 1 5F75672E
 P 7650 3550
+AR Path="/5F75672E" Ref="D201"  Part="1"
+AR Path="/5E73BAE8/5F75672E" Ref="D201"  Part="1"
 F 0 "D201" H 7650 3325 50  0000 C CNN
 F 1 "PS1060L" H 7650 3416 50  0000 C CNN
@@
 	1    0    0    -1
 $EndComp
-$Comp
-L Transistor_FET:CSD18504Q5A Q202
-U 1 1 5F760DD5
-P 7100 4100
-AR Path="/5E73BAE8/5F760DD5" Ref="Q202"  Part="1"
-AR Path="/5E73BB4A/5F760DD5" Ref="Q?"  Part="1"
-F 0 "Q202" H 7306 4146 50  0000 L CNN
-F 1 "VS6412AE" H 7306 4055 50  0000 L CNN
-F 2 "Package_SON:Diodes_PowerDI3333-8" H 7300 4025 50  0001 L CIN
-F 3 "https://datasheet.lcsc.com/szlcsc/1909091006_Vanguard-VS6412AE_C427044.pdf" V 7100 4100 50  0001 L CNN
-	1    7100 4100
-	1    0    0    -1
-$EndComp
-Wire Wire Line
-	7200 3900 7200 3550
-Wire Wire Line
-	6250 3800 6400 3800
+Wire Wire Line
+	6250 3800 6300 3800
 Wire Wire Line
 	4750 3800 6000 3800
-Wire Wire Line
-	6900 4100 6500 4100
-Wire Wire Line
-	6300 4100 6000 4100
-Wire Wire Line
-	6000 4100 6000 3800
 Connection ~ 6000 3800
 Wire Wire Line
 	6000 3800 6050 3800
 Wire Wire Line
-	7200 4300 7200 4450
-Wire Wire Line
-	7200 4450 6950 4450
-Wire Wire Line
-	6700 4450 6950 4450
-Wire Wire Line
 	6700 4200 6700 4450
-Connection ~ 6950 4450
+Wire Wire Line
+	6050 3900 6000 3900
+Wire Wire Line
+	6000 3900 6000 3800
+Wire Wire Line
+	6250 3900 6300 3900
+Wire Wire Line
+	6300 3900 6300 3800
+Connection ~ 6300 3800
+Wire Wire Line
+	6300 3800 6400 3800
 $EndSCHEMATC

Commit message: Layout fertig, Schaltplan erneut checken
Parts:
- removed L301: 22uH PQ2617BHA-220K, Inductor_SMD:PQ2617BHA-330K, symbol Device:L_Small
- added L301: 22uH PQ2617BHA-220K, Inductor_SMD:PQ2617BHA-330K, symbol Device:L_Small_3
Connections:
- wire segments 106 -> 107
Other:
- note removed: "13-39uH"
Changed lines of the file:
@@
 EESchema Schematic File Version 4
-EELAYER 30 0
+LIBS:MukkeBox-cache
+EELAYER 26 0
 EELAYER END
 $Descr A4 11693 8268
@@
 	1    6700 4550
 	-1   0    0    1
-$EndComp
-$Comp
-L Device:L_Small L301
-U 1 1 5E796A70
-P 6700 3300
-F 0 "L301" V 6600 3200 50  0000 L CNN
-F 1 "22uH PQ2617BHA-220K" V 6800 3150 50  0000 L CNN
-F 2 "Inductor_SMD:PQ2617BHA-330K" H 6700 3300 50  0001 C CNN
-F 3 "https://www.mouser.de/datasheet/2/54/bourns_PQ2617BHA_datasheet-1159314.pdf" H 6700 3300 50  0001 C CNN
-	1    6700 3300
-	1    0    0    -1
 $EndComp
 Wire Wire Line
@@
 Text Notes 5800 4600 0    50   ~ 0
 180p
-Text Notes 6950 3450 1    50   ~ 0
-13-39uH
 Text Notes 7950 5550 0    50   ~ 0
 50A
@@
 Wire Wire Line
 	6300 3800 6400 3800
+$Comp
+L Device:L_Small_3 L301
+U 1 1 5EDD1CAF
+P 6700 3300
+F 0 "L301" H 6747 3346 50  0000 L CNN
+F 1 "22uH PQ2617BHA-220K" H 6747 3255 50  0000 L CNN
+F 2 "Inductor_SMD:PQ2617BHA-330K" H 6700 3300 50  0001 C CNN
+F 3 "https://www.mouser.de/datasheet/2/54/bourns_PQ2617BHA_datasheet-1159314.pdf" H 6700 3300 50  0001 C CNN
+	1    6700 3300
+	1    0    0    -1
+$EndComp
+$Comp
+L power:GND #PWR0201
+U 1 1 5EDD85E2
+P 6500 3200
+F 0 "#PWR0201" H 6500 2950 50  0001 C CNN
+F 1 "GND" H 6505 3027 50  0000 C CNN
+F 2 "" H 6500 3200 50  0001 C CNN
+F 3 "" H 6500 3200 50  0001 C CNN
+	1    6500 3200
+	1    0    0    -1
+$EndComp
+Wire Wire Line
+	6650 3200 6500 3200
 $EndSCHEMATC

Commit message: Änderungen von der Arbeit, Viele LCSC Teile für teurere ausgetauscht
Parts:
- added L201: 22uH TAITEC TMPC1265HP-220MG-D, Inductor_SMD:TAITEC TMPC1265HP-220MG-D, symbol Device:L_Small
- L301: symbol Device:L_Small_3 -> MukkeBox-rescue:L_Small_3-Device
- RV_1: footprint Potentiometer_SMD:Potentiometer_Bourns_3314J_Vertical -> Potentiometer_THT:Potentiometer_Bourns_3296W_Vertical
- R_8: value R007 -> R012; footprint Resistor_SMD:R_2010_5025Metric_Pad1.52x2.65mm_HandSolder -> Resistor_SMD:R_2512_6332Metric
Connections:
- wire segments 107 -> 112
Other:
- note added: "alternativ"
Changed lines of the file:
@@
 P 6700 4550
 F 0 "R_8" H 6641 4504 50  0000 R CNN
-F 1 "R007" H 6641 4595 50  0000 R CNN
-F 2 "Resistor_SMD:R_2010_5025Metric_Pad1.52x2.65mm_HandSolder" H 6700 4550 50  0001 C CNN
+F 1 "R012" H 6641 4595 50  0000 R CNN
+F 2 "Resistor_SMD:R_2512_6332Metric" H 6700 4550 50  0001 C CNN
 F 3 "~" H 6700 4550 50  0001 C CNN
 	1    6700 4550
@@
 F 0 "RV_1" H 8880 3846 50  0000 R CNN
 F 1 "10K" H 8880 3755 50  0000 R CNN
-F 2 "Potentiometer_SMD:Potentiometer_Bourns_3314J_Vertical" H 8950 3800 50  0001 C CNN
+F 2 "Potentiometer_THT:Potentiometer_Bourns_3296W_Vertical" H 8950 3800 50  0001 C CNN
 F 3 "https://www.mouser.de/datasheet/2/54/tc33-778219.pdf" H 8950 3800 50  0001 C CNN
 	1    8950 3800
@@
 	5500 2400 6700 2400
 Wire Wire Line
-	6700 2400 6700 3200
+	6700 2400 6700 3100
 Wire Wire Line
 	4750 3500 4800 3500
@@
 Text Notes 5600 4900 0    50   ~ 0
 159p-319p
-Text Notes 6000 3450 0    50   ~ 0
+Text Notes 5650 3900 0    50   ~ 0
 11-13R
 Text Notes 2750 3050 0    50   ~ 0
@@
 	6300 3800 6400 3800
 $Comp
-L Device:L_Small_3 L301
+L MukkeBox-rescue:L_Small_3-Device L301
 U 1 1 5EDD1CAF
 P 6700 3300
+AR Path="/5EDD1CAF" Ref="L301"  Part="1"
+AR Path="/5E73BAE8/5EDD1CAF" Ref="L301"  Part="1"
 F 0 "L301" H 6747 3346 50  0000 L CNN
 F 1 "22uH PQ2617BHA-220K" H 6747 3255 50  0000 L CNN
@@
 Wire Wire Line
 	6650 3200 6500 3200
+$Comp
+L Device:L_Small L201
+U 1 1 5EFA9CC8
+P 6050 3300
+F 0 "L201" H 6098 3346 50  0000 L CNN
+F 1 "22uH TAITEC TMPC1265HP-220MG-D " V 5950 2950 50  0000 L CNN
+F 2 "Inductor_SMD:TAITEC TMPC1265HP-220MG-D" H 6050 3300 50  0001 C CNN
+F 3 "https://datasheet.lcsc.com/szlcsc/TAITEC-TMPC1265HP-220MG-D_C305224.pdf" H 6050 3300 50  0001 C CNN
+	1    6050 3300
+	1    0    0    -1
+$EndComp
+Wire Wire Line
+	6050 3200 6050 3100
+Wire Wire Line
+	6050 3100 6700 3100
+Connection ~ 6700 3100
+Wire Wire Line
+	6700 3100 6700 3200
+Wire Wire Line
+	6050 3400 6050 3550
+Wire Wire Line
+	6050 3550 6700 3550
+Text Notes 6050 3100 0    50   ~ 0
+alternativ
 $EndSCHEMATC

Commit message: Fast fertig TODO: Connector umverdrahten mit beschriftung
Parts:
- C_5_2: value 560uF 50V -> 560u 50V
- R201, R_201, R_202, R_203: footprint Resistor_SMD:R_0603_1608Metric -> Resistor_SMD:R_0603_1608Metric_Pad1.05x0.95mm_HandSolder
- RV_1: footprint Potentiometer_THT:Potentiometer_Bourns_3296W_Vertical -> Potentiometer_THT:Potentiometer_P250
- R_8: footprint Resistor_SMD:R_2512_6332Metric -> Resistor_SMD:R_2512_6332Metric_Pad1.52x3.35mm_HandSolder
Changed lines of the file:
@@
 F 0 "R_8" H 6641 4504 50  0000 R CNN
 F 1 "R012" H 6641 4595 50  0000 R CNN
-F 2 "Resistor_SMD:R_2512_6332Metric" H 6700 4550 50  0001 C CNN
+F 2 "Resistor_SMD:R_2512_6332Metric_Pad1.52x3.35mm_HandSolder" H 6700 4550 50  0001 C CNN
 F 3 "~" H 6700 4550 50  0001 C CNN
 	1    6700 4550
@@
 F 0 "RV_1" H 8880 3846 50  0000 R CNN
 F 1 "10K" H 8880 3755 50  0000 R CNN
-F 2 "Potentiometer_THT:Potentiometer_Bourns_3296W_Vertical" H 8950 3800 50  0001 C CNN
+F 2 "Potentiometer_THT:Potentiometer_P250" H 8950 3800 50  0001 C CNN
 F 3 "https://www.mouser.de/datasheet/2/54/tc33-778219.pdf" H 8950 3800 50  0001 C CNN
 	1    8950 3800
@@
 AR Path="/5E73BAE8/5E9CBBA9" Ref="C_5_2"  Part="1"
 F 0 "C_5_2" H 3050 2750 50  0000 L CNN
-F 1 "560uF 50V" H 3050 2650 50  0000 L CNN
+F 1 "560u 50V" H 3050 2650 50  0000 L CNN
 F 2 "Capacitor_THT:CP_Radial_D12.5mm_P5.00mm" H 2950 2600 50  0001 C CNN
 F 3 "https://www.mouser.de/datasheet/2/420/United-Chemi-Con-1109128.pdf" H 2950 2600 50  0001 C CNN
@@
 F 0 "R_201" H 3541 2854 50  0000 R CNN
 F 1 "100K" H 3541 2945 50  0000 R CNN
-F 2 "Resistor_SMD:R_0603_1608Metric" H 3600 2900 50  0001 C CNN
+F 2 "Resistor_SMD:R_0603_1608Metric_Pad1.05x0.95mm_HandSolder" H 3600 2900 50  0001 C CNN
 F 3 "~" H 3600 2900 50  0001 C CNN
 	1    3600 2900
@@
 F 0 "R201" H 3191 2854 50  0000 R CNN
 F 1 "100K" H 3191 2945 50  0000 R CNN
-F 2 "Resistor_SMD:R_0603_1608Metric" H 3250 2900 50  0001 C CNN
+F 2 "Resistor_SMD:R_0603_1608Metric_Pad1.05x0.95mm_HandSolder" H 3250 2900 50  0001 C CNN
 F 3 "~" H 3250 2900 50  0001 C CNN
 	1    3250 2900
@@
 F 0 "R_202" H 3841 2854 50  0000 R CNN
 F 1 "100K" H 3841 2945 50  0000 R CNN
-F 2 "Resistor_SMD:R_0603_1608Metric" H 3900 2900 50  0001 C CNN
+F 2 "Resistor_SMD:R_0603_1608Metric_Pad1.05x0.95mm_HandSolder" H 3900 2900 50  0001 C CNN
 F 3 "~" H 3900 2900 50  0001 C CNN
 	1    3900 2900
@@
 F 0 "R_203" H 4141 2854 50  0000 R CNN
 F 1 "100K" H 4141 2945 50  0000 R CNN
-F 2 "Resistor_SMD:R_0603_1608Metric" H 4200 2900 50  0001 C CNN
+F 2 "Resistor_SMD:R_0603_1608Metric_Pad1.05x0.95mm_HandSolder" H 4200 2900 50  0001 C CNN
 F 3 "~" H 4200 2900 50  0001 C CNN
 	1    4200 2900

Commit message: Bauteilwerte verändert
Parts:
- R_3: value 422R -> 1K
Other:
- note added: "0,7V FB"
Changed lines of the file:
@@
 P 8950 4450
 F 0 "R_3" H 8891 4404 50  0000 R CNN
-F 1 "422R" H 8891 4495 50  0000 R CNN
+F 1 "1K" H 8891 4495 50  0000 R CNN
 F 2 "Resistor_SMD:R_0603_1608Metric_Pad1.05x0.95mm_HandSolder" H 8950 4450 50  0001 C CNN
 F 3 "~" H 8950 4450 50  0001 C CNN
@@
 F 1 "TPS40210" H 4350 4324 50  0000 C CNN
 F 2 "Package_SO:MSOP-10-1EP_3x3mm_P0.5mm_EP1.68x1.88mm" H 4300 3800 50  0001 C CNN
-F 3 "" H 4300 3800 50  0001 C CNN
+F 3 "https://www.ti.com/lit/ds/symlink/tps40210.pdf?ts=1591439964953&ref_url=https://www.ti.com/product/TPS40210?utm_source%3Dgoogle&utm_medium=cpc&utm_campaign=app-null-null-GPN_EN-cpc-pf-google-eu&utm_content=TPS40210&ds_k=TPS40210&DCM=yes&gclid=EAIaIQobChMIqenB5v_s6QIVme3tCh1OGAzwEAAYASAAEgJRsvD_BwE&gclsrc=aw.ds" H 4300 3800 50  0001 C CNN
 	1    4300 3800
 	1    0    0    -1
@@
 AR Path="/5EDD1CAF" Ref="L301"  Part="1"
 AR Path="/5E73BAE8/5EDD1CAF" Ref="L301"  Part="1"
-F 0 "L301" H 6747 3346 50  0000 L CNN
-F 1 "22uH PQ2617BHA-220K" H 6747 3255 50  0000 L CNN
+F 0 "L301" V 6900 3200 50  0000 L CNN
+F 1 "22uH PQ2617BHA-220K" V 6800 3200 50  0000 L CNN
 F 2 "Inductor_SMD:PQ2617BHA-330K" H 6700 3300 50  0001 C CNN
 F 3 "https://www.mouser.de/datasheet/2/54/bourns_PQ2617BHA_datasheet-1159314.pdf" H 6700 3300 50  0001 C CNN
@@
 U 1 1 5EFA9CC8
 P 6050 3300
-F 0 "L201" H 6098 3346 50  0000 L CNN
+F 0 "L201" V 6150 3200 50  0000 L CNN
 F 1 "22uH TAITEC TMPC1265HP-220MG-D " V 5950 2950 50  0000 L CNN
 F 2 "Inductor_SMD:TAITEC TMPC1265HP-220MG-D" H 6050 3300 50  0001 C CNN
@@
 Text Notes 6050 3100 0    50   ~ 0
 alternativ
+Text Notes 4200 4650 0    50   ~ 0
+0,7V FB
 $EndSCHEMATC

Commit message: Bereit zur Bestellung
Parts:
- C205: value 100n -> 1u
- D201: symbol MukkeBox-rescue:PS1060L-Device -> MukkeBox-rescue:PS1060L-Device-MukkeBox-rescue
- L301: symbol MukkeBox-rescue:L_Small_3-Device -> MukkeBox-rescue:L_Small_3-Device-MukkeBox-rescue
- R_3: value 1K -> 1K5
- U202: symbol MukkeBox-rescue:StepUp-MySymbols -> MukkeBox-rescue:StepUp-MySymbols-MukkeBox-rescue
- U203: symbol MukkeBox-rescue:TPS40210-MySymbols -> MukkeBox-rescue:TPS40210-MySymbols-MukkeBox-rescue
Connections:
- net STEPUP_DISABLE: now reaches U203.3 (DIS/EN)
- no-connect marks 1 -> 0
Other:
- note removed: "50A"
- note removed: "Softstart 5ms"
Changed lines of the file:
@@
 EESchema Schematic File Version 4
-LIBS:MukkeBox-cache
-EELAYER 26 0
+EELAYER 30 0
 EELAYER END
 $Descr A4 11693 8268
@@
 P 8950 4450
 F 0 "R_3" H 8891 4404 50  0000 R CNN
-F 1 "1K" H 8891 4495 50  0000 R CNN
+F 1 "1K5" H 8891 4495 50  0000 R CNN
 F 2 "Resistor_SMD:R_0603_1608Metric_Pad1.05x0.95mm_HandSolder" H 8950 4450 50  0001 C CNN
 F 3 "~" H 8950 4450 50  0001 C CNN
@@
 	8950 4300 8950 4350
 $Comp
-L MukkeBox-rescue:StepUp-MySymbols U202
+L MukkeBox-rescue:StepUp-MySymbols-MukkeBox-rescue U202
 U 1 1 5FE6AEE3
 P 2600 6450
@@
 Möglichkeit fertigen StepUp aufzusetzen
 $Comp
-L MukkeBox-rescue:TPS40210-MySymbols U203
+L MukkeBox-rescue:TPS40210-MySymbols-MukkeBox-rescue U203
 U 1 1 5EDD3766
 P 4300 3800
@@
 P 3500 3650
 F 0 "C205" V 3300 3600 50  0000 L CNN
-F 1 "100n" V 3400 3600 50  0000 L CNN
+F 1 "1u" V 3400 3600 50  0000 L CNN
 F 2 "Capacitor_SMD:C_0603_1608Metric_Pad1.05x0.95mm_HandSolder" H 3500 3650 50  0001 C CNN
 F 3 "~" H 3500 3650 50  0001 C CNN
@@
 Wire Wire Line
 	4800 2400 5500 2400
-NoConn ~ 3950 3800
-Text Notes 2050 3850 0    50   ~ 0
+Text Notes 1250 4000 0    50   ~ 0
 DIS/EN internal pulldown 1M enables device
 Text Notes 4750 1900 0    50   ~ 0
@@
 Text Notes 9250 4050 0    50   ~ 0
 51K7
-Text Notes 2300 3650 0    50   ~ 0
-Softstart 5ms
 Text Notes 3650 4750 0    50   ~ 0
 18k7
@@
 Text Notes 5800 4600 0    50   ~ 0
 180p
-Text Notes 7950 5550 0    50   ~ 0
-50A
 Text Notes 7600 3200 0    50   ~ 0
 10A
@@
 	8050 3550 8550 3550
 $Comp
-L MukkeBox-rescue:PS1060L-Device D201
+L MukkeBox-rescue:PS1060L-Device-MukkeBox-rescue D201
 U 1 1 5F75672E
 P 7650 3550
@@
 	6300 3800 6400 3800
 $Comp
-L MukkeBox-rescue:L_Small_3-Device L301
+L MukkeBox-rescue:L_Small_3-Device-MukkeBox-rescue L301
 U 1 1 5EDD1CAF
 P 6700 3300
@@
 Text Notes 4200 4650 0    50   ~ 0
 0,7V FB
+Text GLabel 2750 3800 0    50   Input ~ 0
+STEPUP_DISABLE
+Wire Wire Line
+	3950 3800 2750 3800
 $EndSCHEMATC
