File: StepDown.sch (KiCad schematic (older format))
At the start: 17 parts, among them J604 Conn_02x01, Q601 2N7002, Q602 2N7002, Q603 MMBT2222LT1G, U602 LM2596S-ADJ

Commit message: neue schematic fertig zum rewiew. DRC clean
Parts:
- added R604: 47K, Resistor_SMD:R_0603_1608Metric_Pad1.05x0.95mm_HandSolder, symbol Device:R_Small
Connections:
- wire segments 53 -> 54
Other:
- moved on the sheet: R609
Changed lines of the file:
@@
 $Descr A4 11693 8268
 encoding utf-8
-Sheet 8 6
+Sheet 6 6
 Title ""
 Date ""
@@
 	3600 3650 5100 4000
 $Comp
-L power:PWR_FLAG #FLG0602
-U 1 1 5ED2C8B6
-P 8350 3250
-F 0 "#FLG0602" H 8350 3325 50  0001 C CNN
-F 1 "PWR_FLAG" H 8350 3424 50  0000 C CNN
-F 2 "" H 8350 3250 50  0001 C CNN
-F 3 "~" H 8350 3250 50  0001 C CNN
-	1    8350 3250
-	1    0    0    -1
-$EndComp
-$Comp
 L power:+3V3 #PWR0606
 U 1 1 5ED2C931
@@
 Connection ~ 4400 3050
 Wire Wire Line
-	4400 3050 3600 3050
+	4400 3050 3900 3050
 Wire Wire Line
 	4600 3250 4400 3250
@@
 L Device:R_Small R?
 U 1 1 5EE77708
-P 3850 5300
+P 3850 4700
 AR Path="/5EE77708" Ref="R?"  Part="1"
 AR Path="/5ED2496F/5EE77708" Ref="R609"  Part="1"
-F 0 "R609" H 3650 5400 50  0000 C CNN
-F 1 "100K" H 3650 5300 50  0000 C CNN
-F 2 "Resistor_SMD:R_0603_1608Metric_Pad1.05x0.95mm_HandSolder" H 3850 5300 50  0001 C CNN
-F 3 "~" H 3850 5300 50  0001 C CNN
-	1    3850 5300
+F 0 "R609" H 3650 4800 50  0000 C CNN
+F 1 "100K" H 3650 4700 50  0000 C CNN
+F 2 "Resistor_SMD:R_0603_1608Metric_Pad1.05x0.95mm_HandSolder" H 3850 4700 50  0001 C CNN
+F 3 "~" H 3850 4700 50  0001 C CNN
+	1    3850 4700
 	1    0    0    -1
 $EndComp
@@
 Wire Wire Line
 	3700 4450 3850 4450
-Wire Wire Line
-	3850 4450 3850 5000
-Connection ~ 3850 5000
 Wire Wire Line
 	4400 3250 4400 4100
@@
 $EndComp
 Wire Wire Line
-	8750 3250 8350 3250
-Connection ~ 8350 3250
-Wire Wire Line
-	8350 3250 8000 3250
-Wire Wire Line
 	6700 3250 7500 3250
+$Comp
+L Device:R_Small R?
+U 1 1 5F175CD1
+P 3850 5300
+AR Path="/5F175CD1" Ref="R?"  Part="1"
+AR Path="/5ED2496F/5F175CD1" Ref="R604"  Part="1"
+F 0 "R604" H 3650 5400 50  0000 C CNN
+F 1 "47K" H 3650 5300 50  0000 C CNN
+F 2 "Resistor_SMD:R_0603_1608Metric_Pad1.05x0.95mm_HandSolder" H 3850 5300 50  0001 C CNN
+F 3 "~" H 3850 5300 50  0001 C CNN
+	1    3850 5300
+	1    0    0    -1
+$EndComp
+Wire Wire Line
+	3850 5000 3850 4800
+Connection ~ 3850 5000
+Wire Wire Line
+	3850 4600 3850 4450
+Wire Wire Line
+	8000 3250 8750 3250
+$Comp
+L power:PWR_FLAG #FLG0104
+U 1 1 5FE15C0B
+P 3900 3050
+F 0 "#FLG0104" H 3900 3125 50  0001 C CNN
+F 1 "PWR_FLAG" H 3900 3224 50  0000 C CNN
+F 2 "" H 3900 3050 50  0001 C CNN
+F 3 "~" H 3900 3050 50  0001 C CNN
+	1    3900 3050
+	1    0    0    -1
+$EndComp
+Connection ~ 3900 3050
+Wire Wire Line
+	3900 3050 3600 3050
 $EndSCHEMATC

Commit message: module, falls schaltung nicht funktioniert hinzugefügt
Parts:
- added J605: Conn_02x01, Connector_PinHeader_2.54mm:PinHeader_1x02_P2.54mm_Vertical, symbol Connector_Generic:Conn_02x01
- added Q604: 2N7002, Package_TO_SOT_SMD:SOT-23, symbol Transistor_FET:2N7002
- added Q605: FDD4685-F085, Package_TO_SOT_SMD:TO-252-2, symbol Device:Q_NMOS_GSD
- added R605, R623, R624: 100K, Resistor_SMD:R_0603_1608Metric_Pad1.05x0.95mm_HandSolder, symbol Device:R_Small
- added R606: 47K, Resistor_SMD:R_0603_1608Metric_Pad1.05x0.95mm_HandSolder, symbol Device:R_Small
- added R607: 1K, Resistor_SMD:R_0603_1608Metric_Pad1.05x0.95mm_HandSolder, symbol Device:R_Small
- added U603: LM2596_Modul, Module:StepDownModul_LM2596, symbol MySymbols:LM2596_Modul
Connections:
- wire segments 54 -> 80
Other:
- note added: "Falls obige Schaltung nicht funktioniert."
- moved on the sheet: J604

Commit message: TODO: power on detect einfügen
Parts:
- removed C602, C607: 68u, Capacitor_THT:CP_Radial_D6.3mm_P2.50mm, symbol Device:CP1_Small
- removed L601: 22uH 6100-101K-RC, Inductor_THT:L_Radial_D12.0mm_P6.00mm_MuRATA_1900R, symbol Device:L_Core_Ferrite_Small
- removed Q601, Q602, Q604: 2N7002, Package_TO_SOT_SMD:SOT-23, symbol Transistor_FET:2N7002
- removed Q603: MMBT2222LT1G, Package_TO_SOT_SMD:SOT-23, symbol Device:Q_NPN_BEC
- removed Q605: FDD4685-F085, Package_TO_SOT_SMD:TO-252-2, symbol Device:Q_NMOS_GSD
- removed R604, R606, R608: 47K, Resistor_SMD:R_0603_1608Metric_Pad1.05x0.95mm_HandSolder, symbol Device:R_Small
- removed R605, R612, R623, R624: 100K, Resistor_SMD:R_0603_1608Metric_Pad1.05x0.95mm_HandSolder, symbol Device:R_Small
- removed R607, R611: 1K, Resistor_SMD:R_0603_1608Metric_Pad1.05x0.95mm_HandSolder, symbol Device:R_Small
- removed R621: 0R, Resistor_SMD:R_0603_1608Metric_Pad1.05x0.95mm_HandSolder, symbol Device:R_Small
- removed R622: 3K3, Resistor_SMD:R_0603_1608Metric_Pad1.05x0.95mm_HandSolder, symbol Device:R_Small
- removed RV601: 10K, Potentiometer_SMD:Potentiometer_Bourns_3314J_Vertical, symbol Device:R_POT
- removed U602: LM2596S-ADJ, Package_TO_SOT_SMD:TO-263-5_TabPin3, symbol Regulator_Switching:LM2596S-ADJ
- removed U603: LM2596_Modul, Module:StepDownModul_LM2596, symbol MySymbols:LM2596_Modul
- added C602, C607, C608: 100nF, Capacitor_SMD:C_0603_1608Metric_Pad1.05x0.95mm_HandSolder, symbol Device:C_Small
- added C611: 22u, Capacitor_THT:CP_Radial_D6.3mm_P2.50mm, symbol Device:CP1_Small
- added L601: 10u Bourns SRN4018, Inductor_SMD:L_Bourns-SRN4018, symbol Device:L_Small
- added R_FBB601: 22K1, Resistor_SMD:R_0603_1608Metric_Pad1.05x0.95mm_HandSolder, symbol Device:R_Small
- added R_FBT601: 51K, Resistor_SMD:R_0603_1608Metric_Pad1.05x0.95mm_HandSolder, symbol Device:R_Small
- added S_601, S_602: MMBT2222LT1G, Package_TO_SOT_SMD:SOT-23, symbol Device:Q_NPN_BEC
- added U602: TPS560430, Package_TO_SOT_SMD:SOT-23-6_Handsoldering, symbol Regulator_Switching:TPS560430
- C601: value 68u -> 2.2u
- R602, R609: value 100K -> 470K
Connections:
- net labels removed: FB, GND_STPDWN
- wire segments 80 -> 50
Other:
- note removed: "Falls obige Schaltung nicht funktioniert."
- moved on the sheet: J604, R609

Commit message: vor änderungen von der Arbeit
Parts:
- added Q1: 2N7002, Package_TO_SOT_SMD:SOT-23, symbol Transistor_FET:2N7002
- added R1: 100K, Resistor_SMD:R_0603_1608Metric_Pad1.05x0.95mm_HandSolder, symbol Device:R_Small
- added R2: 47K, Resistor_SMD:R_0603_1608Metric_Pad1.05x0.95mm_HandSolder, symbol Device:R_Small
- added R3: 10K, Resistor_SMD:R_0603_1608Metric_Pad1.05x0.95mm_HandSolder, symbol Device:R_Small
- U602: symbol Regulator_Switching:TPS560430 -> MukkeBox-rescue:TPS560430-Regulator_Switching
Connections:
- net labels added: 3V3_ENABLED
- wire segments 50 -> 56
Changed lines of the file:
@@
 	9000 3200 8250 3200
 $Comp
-L Regulator_Switching:TPS560430 U602
+L MukkeBox-rescue:TPS560430-Regulator_Switching U602
 U 1 1 5ECDAABE
 P 5950 3150
@@
 F 1 "TPS560430" H 5950 3384 50  0000 C CNN
 F 2 "Package_TO_SOT_SMD:SOT-23-6_Handsoldering" H 5150 2750 50  0001 L CNN
-F 3 "http://www.ti.com/lit/ds/symlink/tps560200.pdf" H 5700 2800 50  0001 C CNN
+F 3 "https://www.ti.com/lit/ds/symlink/tps560430.pdf?ts=1590476433528" H 5700 2800 50  0001 C CNN
 	1    5950 3150
 	1    0    0    -1
@@
 Wire Wire Line
 	4500 3050 5650 3050
+$Comp
+L power:GND #PWR?
+U 1 1 5ED4AAC5
+P 6700 2400
+AR Path="/5E73BB4A/5ED4AAC5" Ref="#PWR?"  Part="1"
+AR Path="/5ED2496F/5ED4AAC5" Ref="#PWR01"  Part="1"
+F 0 "#PWR01" H 6700 2150 50  0001 C CNN
+F 1 "GND" H 6705 2227 50  0000 C CNN
+F 2 "" H 6700 2400 50  0001 C CNN
+F 3 "" H 6700 2400 50  0001 C CNN
+	1    6700 2400
+	1    0    0    -1
+$EndComp
+$Comp
+L Device:R_Small R?
+U 1 1 5ED4AACB
+P 6700 1850
+AR Path="/5E73BB4A/5ED4AACB" Ref="R?"  Part="1"
+AR Path="/5ED2496F/5ED4AACB" Ref="R1"  Part="1"
+F 0 "R1" H 6759 1896 50  0000 L CNN
+F 1 "100K" H 6759 1805 50  0000 L CNN
+F 2 "Resistor_SMD:R_0603_1608Metric_Pad1.05x0.95mm_HandSolder" H 6700 1850 50  0001 C CNN
+F 3 "~" H 6700 1850 50  0001 C CNN
+	1    6700 1850
+	1    0    0    -1
+$EndComp
+$Comp
+L Device:R_Small R?
+U 1 1 5ED4AAD1
+P 6700 2300
+AR Path="/5E73BB4A/5ED4AAD1" Ref="R?"  Part="1"
+AR Path="/5ED2496F/5ED4AAD1" Ref="R2"  Part="1"
+F 0 "R2" H 6759 2346 50  0000 L CNN
+F 1 "47K" H 6759 2255 50  0000 L CNN
+F 2 "Resistor_SMD:R_0603_1608Metric_Pad1.05x0.95mm_HandSolder" H 6700 2300 50  0001 C CNN
+F 3 "~" H 6700 2300 50  0001 C CNN
+	1    6700 2300
+	1    0    0    -1
+$EndComp
+$Comp
+L power:+3V3 #PWR?
+U 1 1 5ED4AAD7
+P 7200 1650
+AR Path="/5E73BB4A/5ED4AAD7" Ref="#PWR?"  Part="1"
+AR Path="/5ED2496F/5ED4AAD7" Ref="#PWR02"  Part="1"
+F 0 "#PWR02" H 7200 1500 50  0001 C CNN
+F 1 "+3V3" H 7215 1823 50  0000 C CNN
+F 2 "" H 7200 1650 50  0001 C CNN
+F 3 "" H 7200 1650 50  0001 C CNN
+	1    7200 1650
+	1    0    0    -1
+$EndComp
+$Comp
+L Device:R_Small R?
+U 1 1 5ED4AADD
+P 7200 1750
+AR Path="/5E73BB4A/5ED4AADD" Ref="R?"  Part="1"
+AR Path="/5ED2496F/5ED4AADD" Ref="R3"  Part="1"
+F 0 "R3" H 7259 1796 50  0000 L CNN
+F 1 "10K" H 7259 1705 50  0000 L CNN
+F 2 "Resistor_SMD:R_0603_1608Metric_Pad1.05x0.95mm_HandSolder" H 7200 1750 50  0001 C CNN
+F 3 "~" H 7200 1750 50  0001 C CNN
+	1    7200 1750
+	1    0    0    -1
+$EndComp
+Text GLabel 7450 1850 2    50   Input ~ 0
+3V3_ENABLED
+Wire Wire Line
+	7450 1850 7200 1850
+Connection ~ 7200 1850
+$Comp
+L Transistor_FET:2N7002 Q?
+U 1 1 5ED4AAE6
+P 7100 2050
+AR Path="/5E73BB4A/5ED4AAE6" Ref="Q?"  Part="1"
+AR Path="/5ED2496F/5ED4AAE6" Ref="Q1"  Part="1"
+F 0 "Q1" H 7305 2096 50  0000 L CNN
+F 1 "2N7002" H 7305 2005 50  0000 L CNN
+F 2 "Package_TO_SOT_SMD:SOT-23" H 7300 1975 50  0001 L CIN
+F 3 "https://www.fairchildsemi.com/datasheets/2N/2N7002.pdf" H 7100 2050 50  0001 L CNN
+	1    7100 2050
+	1    0    0    -1
+$EndComp
+Wire Wire Line
+	6900 2050 6700 2050
+Wire Wire Line
+	6700 2050 6700 1950
+Wire Wire Line
+	6700 2200 6700 2050
+Connection ~ 6700 2050
+$Comp
+L power:GND #PWR?
+U 1 1 5ED4AAF0
+P 7200 2400
+AR Path="/5E73BB4A/5ED4AAF0" Ref="#PWR?"  Part="1"
+AR Path="/5ED2496F/5ED4AAF0" Ref="#PWR03"  Part="1"
+F 0 "#PWR03" H 7200 2150 50  0001 C CNN
+F 1 "GND" H 7205 2227 50  0000 C CNN
+F 2 "" H 7200 2400 50  0001 C CNN
+F 3 "" H 7200 2400 50  0001 C CNN
+	1    7200 2400
+	1    0    0    -1
+$EndComp
+Wire Wire Line
+	7200 2400 7200 2250
+Wire Wire Line
+	6700 1750 6700 1600
+Text GLabel 6700 1600 0    50   Input ~ 0
+3V3_EN
 $EndSCHEMATC

Commit message: Charger ausgetauscht, Mosfet und Dioden durch billigere ersetzt
Parts:
- removed S_601, S_602: MMBT2222LT1G, Package_TO_SOT_SMD:SOT-23, symbol Device:Q_NPN_BEC
- added D601: BAT54C, Package_TO_SOT_SMD:SOT-23, symbol Diode:BAT54C
Connections:
- wire segments 56 -> 49
Changed lines of the file:
@@
 EESchema Schematic File Version 4
-EELAYER 30 0
+LIBS:MukkeBox-cache
+EELAYER 26 0
 EELAYER END
 $Descr A4 11693 8268
@@
 	1    0    0    -1
 $EndComp
-Text Label 4850 2500 0    50   ~ 0
+Text Label 4950 2500 2    50   ~ 0
 3V3_ON_OFF
-Text GLabel 5500 1600 0    50   Input ~ 0
+Text GLabel 5650 1600 0    50   Input ~ 0
 3V3_EN
 $Comp
@@
 	3350 3050 3900 3050
 Wire Wire Line
-	5650 2250 5650 2500
-Wire Wire Line
-	4550 2500 4550 2250
-Wire Wire Line
 	5050 3200 5400 3200
-Text GLabel 4400 1600 0    50   Input ~ 0
+Text GLabel 5050 1600 0    50   Input ~ 0
 DC_20V_POWER_SUPPLY
-Wire Wire Line
-	4400 1600 4550 1600
-Wire Wire Line
-	5500 1600 5650 1600
 $Comp
 L Device:C_Small C?
@@
 	5400 3750 5550 3750
 Wire Wire Line
-	4550 2500 5400 2500
+	4950 2500 5400 2500
 $Comp
 L Device:R_Small R?
@@
 	5400 2700 5400 2500
 Connection ~ 5400 2500
-Wire Wire Line
-	5400 2500 5650 2500
 $Comp
 L power:PWR_FLAG #FLG0107
@@
 Text GLabel 6700 1600 0    50   Input ~ 0
 3V3_EN
-Wire Wire Line
-	5650 1600 5650 1850
-Wire Wire Line
-	4550 1600 4550 1850
-Wire Wire Line
-	5350 1850 5650 1850
-Wire Wire Line
-	5350 2050 5350 1850
-Wire Wire Line
-	4250 2050 4250 1850
-Wire Wire Line
-	4250 1850 4550 1850
-Connection ~ 4550 1850
-$Comp
-L Device:Q_NPN_BEC S_?
-U 1 1 5ED0F92E
-P 4450 2050
-AR Path="/5E73BAE8/5ED0F92E" Ref="S_?"  Part="1"
-AR Path="/5ED2496F/5ED0F92E" Ref="S_601"  Part="1"
-F 0 "S_601" H 4640 2096 50  0000 L CNN
-F 1 "MMBT2222LT1G" H 4640 2005 50  0000 L CNN
-F 2 "Package_TO_SOT_SMD:SOT-23" H 4650 2150 50  0001 C CNN
-F 3 "https://www.mouser.de/datasheet/2/308/MMBT2222LT1-D-1811600.pdf" H 4450 2050 50  0001 C CNN
-	1    4450 2050
-	1    0    0    -1
-$EndComp
-Connection ~ 5650 1850
-$Comp
-L Device:Q_NPN_BEC S_?
-U 1 1 5ED128E5
-P 5550 2050
-AR Path="/5E73BAE8/5ED128E5" Ref="S_?"  Part="1"
-AR Path="/5ED2496F/5ED128E5" Ref="S_602"  Part="1"
-F 0 "S_602" H 5740 2096 50  0000 L CNN
-F 1 "MMBT2222LT1G" H 5740 2005 50  0000 L CNN
-F 2 "Package_TO_SOT_SMD:SOT-23" H 5750 2150 50  0001 C CNN
-F 3 "https://www.mouser.de/datasheet/2/308/MMBT2222LT1-D-1811600.pdf" H 5550 2050 50  0001 C CNN
-	1    5550 2050
-	1    0    0    -1
-$EndComp
+$Comp
+L Diode:BAT54C D?
+U 1 1 5F7DF8E3
+P 5400 2300
+AR Path="/5E73BB4A/5F7DF8E3" Ref="D?"  Part="1"
+AR Path="/5ED2496F/5F7DF8E3" Ref="D601"  Part="1"
+F 0 "D601" H 5400 2525 50  0000 C CNN
+F 1 "BAT54C" H 5400 2434 50  0000 C CNN
+F 2 "Package_TO_SOT_SMD:SOT-23" H 5475 2425 50  0001 L CNN
+F 3 "http://www.diodes.com/_files/datasheets/ds11005.pdf" H 5320 2300 50  0001 C CNN
+	1    5400 2300
+	1    0    0    -1
+$EndComp
+Wire Wire Line
+	5050 1600 5100 1600
+Wire Wire Line
+	5100 1600 5100 2300
+Wire Wire Line
+	5650 1600 5700 1600
+Wire Wire Line
+	5700 1600 5700 2300
 $EndSCHEMATC

Commit message: Änderungen Arbeit hinzugefügt: Layout neuer Charger
Parts:
- R_FBB601: value 22K1 -> 20K
- R_FBT601: value 51K -> 47K
Other:
- note added: "22K1"
- note added: "51K"
Changed lines of the file:
@@
 EESchema Schematic File Version 4
-LIBS:MukkeBox-cache
-EELAYER 26 0
+EELAYER 30 0
 EELAYER END
 $Descr A4 11693 8268
@@
 AR Path="/5ED2496F/5ECED53D" Ref="R_FBT601"  Part="1"
 F 0 "R_FBT601" H 7050 3400 50  0000 C CNN
-F 1 "51K" H 7050 3300 50  0000 C CNN
+F 1 "47K" H 7050 3300 50  0000 C CNN
 F 2 "Resistor_SMD:R_0603_1608Metric_Pad1.05x0.95mm_HandSolder" H 7250 3300 50  0001 C CNN
 F 3 "~" H 7250 3300 50  0001 C CNN
@@
 AR Path="/5ED2496F/5ECED695" Ref="R_FBB601"  Part="1"
 F 0 "R_FBB601" H 7050 3700 50  0000 C CNN
-F 1 "22K1" H 7050 3600 50  0000 C CNN
+F 1 "20K" H 7050 3600 50  0000 C CNN
 F 2 "Resistor_SMD:R_0603_1608Metric_Pad1.05x0.95mm_HandSolder" H 7250 3600 50  0001 C CNN
 F 3 "~" H 7250 3600 50  0001 C CNN
@@
 Wire Wire Line
 	5700 1600 5700 2300
+Text Notes 7050 3350 0    50   ~ 0
+51K
+Text Notes 7000 3650 0    50   ~ 0
+22K1
 $EndSCHEMATC
