File: _autosave-MukkeBox.kicad_pcb (KiCad board)
At the start: 2 copper layers, 200 x 105 mm, 278 parts, among them J101 Conn_02x20_Odd_Even, J102 Conn_01x04, J103 Conn_02x05_Odd_Even, J104 Conn_02x05_Odd_Even, J301 Conn_02x04_Odd_Even, J302 Conn_02x04_Odd_Even, J303 TB001-500-04BE CUI_Devices, J401 TB001-500-02BE CUI_Devices, J501 TB001-500-04BE CUI_Devices, J601 Conn_01x03_Female, J602 Conn_02x01, J603 Conn_02x06_Odd_Even, J604 Conn_02x01, J605 Conn_02x01, Q1 2N7002, Q201 VS6412AE, Q301 2N7002, Q302 HSBB3103, Q303 2N7002, Q304 HSBB3103, Q305 VS6412AE, Q306 2N7002, Q307 BSS84, Q308 2N7002, Q309 VS6412AE, Q310 HSBB3103, Q311 HSBB3103, Q501 2N7002, SW501 DS04-254-2-02BK-SMT, U101 LM35-LP, U102 STM32F030C6Tx_MukkeBox, U103 MCP9700, U202 StepUp, U203 TPS40210, U301 BQ24610, U501 TDA7498L, U502 BK8000L, U503 TDA7719, U504 AP2553AW6-7, U505 JW5026, U602 JW5026, Y101 FOXSDLF/080-20

Commit message: Bestellung abgeschickt
Parts:
- R313: value 470K -> 100K
- R314: value 47K -> 10K
- R413: value 47K -> 100K
Changed lines of the file:
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@@
       (effects (font (size 1 1) (thickness 0.15)))
     )
-    (fp_text value 470K (at 0 1.43 90) (layer F.Fab)
+    (fp_text value 100K (at 0 1.43 90) (layer F.Fab)
       (effects (font (size 1 1) (thickness 0.15)))
     )
@@
       (effects (font (size 0.8 0.8) (thickness 0.15)))
     )
-    (fp_text value 47K (at 0 1.43 90) (layer F.Fab)
+    (fp_text value 10K (at 0 1.43 90) (layer F.Fab)
       (effects (font (size 1 1) (thickness 0.15)))
     )
@@
       (effects (font (size 1 1) (thickness 0.15)))
     )
-    (fp_text value 47K (at 0 1.43 270) (layer F.Fab)
-      (effects (font (size 1 1) (thickness 0.15)))
-    )
+    (fp_text value 100K (at 0 1.43 270) (layer F.Fab)
+      (effects (font (size 1 1) (thickness 0.15)))
+    )
