File: MukkeBox.kicad_pcb (KiCad board)
At the start: 2 copper layers, 200 x 105 mm, 275 parts, among them J101 Conn_02x20_Odd_Even, J102 Conn_01x04, J103 Conn_02x05_Odd_Even, J104 Conn_02x05_Odd_Even, J301 Conn_02x04_Odd_Even, J302 Conn_02x04_Odd_Even, J303 TB001-500-04BE CUI_Devices, J401 TB001-500-02BE CUI_Devices, J501 TB001-500-04BE CUI_Devices, J601 Conn_01x03_Female, J602 Conn_02x01, J603 Conn_02x06_Odd_Even, J604 Conn_02x01, J605 Conn_02x01, Q1 2N7002, Q201 VS6412AE, Q301 2N7002, Q302 HSBB3103, Q303 2N7002, Q304 HSBB3103, Q305 VS6412AE, Q306 2N7002, Q307 BSS84, Q308 2N7002, Q309 VS6412AE, Q310 HSBB3103, Q311 HSBB3103, Q501 2N7002, SW501 DS04-254-2-02BK-SMT, U101 LM35-LP, U102 STM32F030C6Tx_MukkeBox, U103 MCP9700, U202 StepUp, U203 TPS40210, U301 BQ24610, U501 TDA7498L, U502 BK8000L, U503 TDA7719, U504 AP2553AW6-7, U505 JW5026, U602 JW5026, Y101 FOXSDLF/080-20

Commit message: Fast fertig TODO: Connector umverdrahten mit beschriftung
Parts:
- added R309: 100K, Resistor_SMD:R_0603_1608Metric_Pad1.05x0.95mm_HandSolder, F.Cu at (68.7, 49.8)
- added REF**: WEEE-Logo_4.2x6mm_SilkScreen, Symbol:WEEE-Logo_4.2x6mm_SilkScreen, F.Cu at (215.8, 44.8)
- added REF**: KiCAD Logo, Symbol:Symbol_KiCAD-Logo_CopperAndSilkScreenTop, F.Cu at (225.7, 45.5)
- C101, C102, C103, C106, C107, C108, C109, C114, C115, C501, C502, C504, C505, C506, C510, C541, C543, C544, C602, C607, C608, C612: value 100nF -> 100n
- C104, C105: value 20pF -> 20p
- C110, C111, C112, C113: value 10nF -> 10n
- C411: footprint Capacitor_THT:CP_Radial_D6.3mm_P2.50mm -> Capacitor_THT:CP_Radial_D4.0mm_P2.00mm
- C503: value 2.2u -> 10u; footprint Capacitor_THT:CP_Radial_D4.0mm_P1.50mm -> Capacitor_THT:CP_Radial_D4.0mm_P2.00mm
- C507, C517, C518, C534: value 1nF -> 1n
- C508, C509, C536: footprint Capacitor_THT:CP_Radial_D4.0mm_P1.50mm -> Capacitor_THT:CP_Radial_D4.0mm_P2.00mm
- C511, C512: value 100nF -> 100n; footprint Capacitor_SMD:C_1210_3225Metric -> Capacitor_SMD:C_0603_1608Metric_Pad1.05x0.95mm_HandSolder
- C514, C515: value 1uF -> 2.2u
- C519, C520: value 470nF -> 470n
- C521, C522, C523, C524, C526, C527, C528, C529: value 220nF -> 220n
- C525: value 560uF 50V -> 560u 50V; footprint Capacitor_THT:CP_Radial_D13.0mm_P5.00mm -> Capacitor_THT:CP_Radial_D12.5mm_P5.00mm
- C530, C531, C532, C_5_2: value 560uF 50V -> 560u 50V
- C542: footprint Capacitor_THT:CP_Radial_D5.0mm_P2.50mm -> Capacitor_THT:CP_Radial_D4.0mm_P2.00mm
- C601: value 2.2u -> 10u; footprint Capacitor_THT:CP_Radial_D6.3mm_P2.50mm -> Capacitor_THT:CP_Radial_D4.0mm_P2.00mm
- C611: value 22u -> 10u; footprint Capacitor_THT:CP_Radial_D6.3mm_P2.50mm -> Capacitor_THT:CP_Radial_D4.0mm_P2.00mm
- R19C301, R306: value 100K -> 1K
- R201, R_201, R_202, R_203: footprint Resistor_SMD:R_0603_1608Metric -> Resistor_SMD:R_0603_1608Metric_Pad1.05x0.95mm_HandSolder
- R505: value 100k -> 100K
- RV_1: footprint Potentiometer_THT:Potentiometer_Bourns_3296W_Vertical -> Potentiometer_THT:Potentiometer_P250
- R_8: footprint Resistor_SMD:R_2512_6332Metric -> Resistor_SMD:R_2512_6332Metric_Pad1.52x3.35mm_HandSolder
- moved R101 9.50 mm to (119.1, 121.5), turned to 0 degrees
- moved R102 7.40 mm to (119.1, 123.1), turned to 0 degrees
- moved C411 2.20 mm to (78.6, 68.3)
- moved J103 1.24 mm to (50.4, 120.1)
- moved J604 1.12 mm to (50.4, 114.0), turned to 90 degrees
- moved C515 0.75 mm to (205.6, 75.0)
- moved C514 0.62 mm to (194.4, 75.0)
- moved R_8 0.60 mm to (126.6, 93.4)
- moved C508 0.36 mm to (230.4, 118.9)
- moved C512 0.36 mm to (205.6, 77.5)
- moved J401 0.35 mm to (50.1, 54.6)
- moved C511 0.12 mm to (194.4, 77.1)
- moved U101 0.07 mm to (129.3, 136.0)
Connections:
- C305 pad 2: /00_Charger/TS -> Net-(C305-Pad2)
- U301 pad 6: /00_Charger/TS -> Net-(C305-Pad2)
- U502 pad 17: Net-(U502-Pad17) -> GNDA
Routing:
- net /I2C1_SDA: track 35.1 -> 43.5 mm
- net Net-(C305-Pad2): track 0.00 -> 8.30 mm
- net /I2C1_SCL: track 38.5 -> 43.6 mm
- net /00_Charger/TS: track 57.4 -> 53.2 mm
- net GNDA: track 115.4 -> 118.1 mm, vias 19 -> 20
- net /SWDIO: track 51.0 -> 49.3 mm
- net /RST: track 39.7 -> 38.4 mm
- net +3V3: track 352.3 -> 351.1 mm
- net CHARGER_STAT2: track 78.7 -> 79.8 mm
- net /ST_Link_3V3: track 55.5 -> 54.5 mm
- net /SWCLK: track 49.2 -> 48.2 mm
- net TxR: track 83.0 -> 84.0 mm
- net Net-(Q201-Pad1): track 9.28 -> 10.2 mm
- net RxT: track 85.6 -> 86.4 mm
- net Net-(C611-Pad1): track 15.1 -> 14.4 mm
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Other:
- board text added: "3V3"
- board text added: "3V3_ext"
- board text added: "GND"
- board text added: "GurkiBox V0.2"
- board text added: "Mute :("
- board text added: "RST"
- board text added: "RX"
- board text added: "SCL"
- board text added: "SDA"
- board text added: "SWCLK"
- board text added: "SWDIO"
- board text added: "TX"

Commit message: Bestellung abgeschickt
Parts:
- R313: value 470K -> 100K
- R314: value 47K -> 10K
- R413: value 47K -> 100K
Changed lines of the file:
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@@
     (tags "capacitor handsolder")
     (attr smd)
-    (fp_text reference C110 (at 0 -2.6 180) (layer F.SilkS)
+    (fp_text reference C110 (at -0.2 1.3 270) (layer F.SilkS)
       (effects (font (size 1 1) (thickness 0.15)))
     )
@@
     (tags "capacitor handsolder")
     (attr smd)
-    (fp_text reference C111 (at 0 2.7 180) (layer F.SilkS)
+    (fp_text reference C111 (at 0.1 -1.4 270) (layer F.SilkS)
       (effects (font (size 1 1) (thickness 0.15)))
     )
@@
     (tags "resistor handsolder")
     (attr smd)
-    (fp_text reference R119 (at 0 2.7 180) (layer F.SilkS)
+    (fp_text reference R119 (at -0.1 -1.4 270) (layer F.SilkS)
       (effects (font (size 1 1) (thickness 0.15)))
     )
@@
     (tags "resistor handsolder")
     (attr smd)
-    (fp_text reference R120 (at -0.1 2.7) (layer F.SilkS)
+    (fp_text reference R120 (at -0.1 -1.4 90) (layer F.SilkS)
       (effects (font (size 1 1) (thickness 0.15)))
     )
@@
       (effects (font (size 1 1) (thickness 0.15)))
     )
-    (fp_text value 470K (at 0 1.43 90) (layer F.Fab)
+    (fp_text value 100K (at 0 1.43 90) (layer F.Fab)
       (effects (font (size 1 1) (thickness 0.15)))
     )
@@
       (effects (font (size 0.8 0.8) (thickness 0.15)))
     )
-    (fp_text value 47K (at 0 1.43 90) (layer F.Fab)
+    (fp_text value 10K (at 0 1.43 90) (layer F.Fab)
       (effects (font (size 1 1) (thickness 0.15)))
     )
@@
       (effects (font (size 1 1) (thickness 0.15)))
     )
-    (fp_text value 47K (at 0 1.43 270) (layer F.Fab)
+    (fp_text value 100K (at 0 1.43 270) (layer F.Fab)
       (effects (font (size 1 1) (thickness 0.15)))
     )
